File: MainBoard/Main board schematic.sch (EAGLE design)
At the start: 16 parts

Commit message: CIrcuit for switches
Seperate schematic for switches (Updated)
Parts:
- added BUTTON_1, BUTTON_10, BUTTON_11, BUTTON_12, BUTTON_13, BUTTON_14, BUTTON_15, BUTTON_16, BUTTON_2, BUTTON_3, BUTTON_4, BUTTON_5, BUTTON_6, BUTTON_7, BUTTON_8, BUTTON_9: CT10-XXXX-A2, switch-coto:CT10-XXXX-A2
- added C10, C11, C12, C13, C14, C15, C16, C17, C2, C3, C4, C5, C6, C7, C8, C9: (no value), capacitor-wima:C5/3
- added IC1, IC10, IC12, IC13, IC14, IC16, IC17, IC18, IC2, IC20, IC21, IC22, IC24, IC25, IC26, IC28, IC29, IC30, IC32, IC33, IC34, IC36, IC37, IC38, IC4, IC40, IC41, IC42, IC44, IC45, IC46, IC48, IC49, IC5, IC50, IC52, IC53, IC54, IC56, IC57, IC58, IC6, IC60, IC61, IC62, IC64, IC8, IC9: 4042D, 40xx:4042D
- added IC11, IC15, IC19, IC23, IC27, IC3, IC31, IC35, IC39, IC43, IC47, IC51, IC55, IC59, IC63, IC7: 4081D, 40xx:4081D
- added R1, R10, R11, R12, R13, R14, R15, R16, R17, R18, R19, R2, R20, R21, R22, R23, R24, R25, R26, R27, R28, R29, R3, R30, R31, R32, R4, R5, R6, R7, R8, R9: 1K, rcl:R-US_0204/7
Connections:
- new net CLK: IC10A.CLK, IC12A.CLK, IC13A.CLK, IC14A.CLK, IC16A.CLK, IC17A.CLK, IC18A.CLK, IC1A.CLK, IC20A.CLK, IC21A.CLK, IC22A.CLK, IC24A.CLK, IC25A.CLK, IC26A.CLK, IC28A.CLK, IC29A.CLK, IC2A.CLK, IC30A.CLK, IC32A.CLK, IC33A.CLK, IC34A.CLK, IC36A.CLK, IC37A.CLK, IC38A.CLK, IC40A.CLK, IC41A.CLK, IC42A.CLK, IC44A.CLK, IC45A.CLK, IC46A.CLK, IC48A.CLK, IC49A.CLK, IC4A.CLK, IC50A.CLK, IC52A.CLK, IC53A.CLK, IC54A.CLK, IC56A.CLK, IC57A.CLK, IC58A.CLK, IC5A.CLK, IC60A.CLK, IC61A.CLK, IC62A.CLK, IC64A.CLK, IC6A.CLK, IC8A.CLK, IC9A.CLK
- new net N$100: IC38A.!Q0, IC38A.!Q1, IC38A.!Q2, IC38A.!Q3, IC40A.D0, IC40A.D1, IC40A.D2, IC40A.D3, IC40A.POL
- new net N$101: IC38A.Q0, IC38A.Q1, IC38A.Q2, IC38A.Q3, IC39A.I0
- new net N$102: BUTTON_10.1
- new net N$103: BUTTON_11.2, R21.1
- new net N$104: C12.1, IC41A.D0, IC41A.D1, IC41A.D2, IC41A.D3, IC41A.POL, R21.2, R22.2
- new net N$105: IC41A.Q0, IC41A.Q1, IC41A.Q2, IC41A.Q3, IC42A.D0, IC42A.D1, IC42A.D2, IC42A.D3, IC42A.POL
- new net N$106: IC43A.I1, IC44A.Q0, IC44A.Q1, IC44A.Q2, IC44A.Q3
- new net N$107: IC42A.!Q0, IC42A.!Q1, IC42A.!Q2, IC42A.!Q3, IC44A.D0, IC44A.D1, IC44A.D2, IC44A.D3, IC44A.POL
- new net N$108: IC42A.Q0, IC42A.Q1, IC42A.Q2, IC42A.Q3, IC43A.I0
- new net N$109: BUTTON_11.1
- new net N$110: BUTTON_12.2, R23.1
- new net N$111: C13.1, IC45A.D0, IC45A.D1, IC45A.D2, IC45A.D3, IC45A.POL, R23.2, R24.2
- new net N$112: IC45A.Q0, IC45A.Q1, IC45A.Q2, IC45A.Q3, IC46A.D0, IC46A.D1, IC46A.D2, IC46A.D3, IC46A.POL
- new net N$113: IC47A.I1, IC48A.Q0, IC48A.Q1, IC48A.Q2, IC48A.Q3
- new net N$114: IC46A.!Q0, IC46A.!Q1, IC46A.!Q2, IC46A.!Q3, IC48A.D0, IC48A.D1, IC48A.D2, IC48A.D3, IC48A.POL
- new net N$115: IC46A.Q0, IC46A.Q1, IC46A.Q2, IC46A.Q3, IC47A.I0
- new net N$116: BUTTON_12.1
- new net N$117: BUTTON_13.2, R25.1
- new net N$118: C14.1, IC49A.D0, IC49A.D1, IC49A.D2, IC49A.D3, IC49A.POL, R25.2, R26.2
- new net N$119: IC49A.Q0, IC49A.Q1, IC49A.Q2, IC49A.Q3, IC50A.D0, IC50A.D1, IC50A.D2, IC50A.D3, IC50A.POL
- new net N$120: IC51A.I1, IC52A.Q0, IC52A.Q1, IC52A.Q2, IC52A.Q3
- new net N$121: IC50A.!Q0, IC50A.!Q1, IC50A.!Q2, IC50A.!Q3, IC52A.D0, IC52A.D1, IC52A.D2, IC52A.D3, IC52A.POL
- new net N$122: IC50A.Q0, IC50A.Q1, IC50A.Q2, IC50A.Q3, IC51A.I0
- new net N$123: BUTTON_13.1
- new net N$124: BUTTON_14.2, R27.1
- new net N$125: C15.1, IC53A.D0, IC53A.D1, IC53A.D2, IC53A.D3, IC53A.POL, R27.2, R28.2
- new net N$126: IC53A.Q0, IC53A.Q1, IC53A.Q2, IC53A.Q3, IC54A.D0, IC54A.D1, IC54A.D2, IC54A.D3, IC54A.POL
- new net N$127: IC55A.I1, IC56A.Q0, IC56A.Q1, IC56A.Q2, IC56A.Q3
- new net N$128: IC54A.!Q0, IC54A.!Q1, IC54A.!Q2, IC54A.!Q3, IC56A.D0, IC56A.D1, IC56A.D2, IC56A.D3, IC56A.POL
- new net N$129: IC54A.Q0, IC54A.Q1, IC54A.Q2, IC54A.Q3, IC55A.I0
- new net N$130: BUTTON_14.1
- new net N$131: BUTTON_15.2, R29.1
- new net N$132: C16.1, IC57A.D0, IC57A.D1, IC57A.D2, IC57A.D3, IC57A.POL, R29.2, R30.2
- new net N$133: IC57A.Q0, IC57A.Q1, IC57A.Q2, IC57A.Q3, IC58A.D0, IC58A.D1, IC58A.D2, IC58A.D3, IC58A.POL
- new net N$134: IC59A.I1, IC60A.Q0, IC60A.Q1, IC60A.Q2, IC60A.Q3
- new net N$135: IC58A.!Q0, IC58A.!Q1, IC58A.!Q2, IC58A.!Q3, IC60A.D0, IC60A.D1, IC60A.D2, IC60A.D3, IC60A.POL
- new net N$136: IC58A.Q0, IC58A.Q1, IC58A.Q2, IC58A.Q3, IC59A.I0
- new net N$137: BUTTON_15.1
- new net N$138: BUTTON_16.2, R31.1
- new net N$139: C17.1, IC61A.D0, IC61A.D1, IC61A.D2, IC61A.D3, IC61A.POL, R31.2, R32.2
- new net N$140: IC61A.Q0, IC61A.Q1, IC61A.Q2, IC61A.Q3, IC62A.D0, IC62A.D1, IC62A.D2, IC62A.D3, IC62A.POL
- new net N$141: IC63A.I1, IC64A.Q0, IC64A.Q1, IC64A.Q2, IC64A.Q3
- new net N$142: IC62A.!Q0, IC62A.!Q1, IC62A.!Q2, IC62A.!Q3, IC64A.D0, IC64A.D1, IC64A.D2, IC64A.D3, IC64A.POL
- new net N$143: IC62A.Q0, IC62A.Q1, IC62A.Q2, IC62A.Q3, IC63A.I0
- new net N$144: BUTTON_16.1
- new net N$20: BUTTON_2.2, R2.1
- new net N$21: C3.1, IC5A.D0, IC5A.D1, IC5A.D2, IC5A.D3, IC5A.POL, R2.2, R3.2
- new net N$31: IC5A.Q0, IC5A.Q1, IC5A.Q2, IC5A.Q3, IC6A.D0, IC6A.D1, IC6A.D2, IC6A.D3, IC6A.POL
- new net N$37: IC7A.I1, IC8A.Q0, IC8A.Q1, IC8A.Q2, IC8A.Q3
- new net N$38: IC6A.!Q0, IC6A.!Q1, IC6A.!Q2, IC6A.!Q3, IC8A.D0, IC8A.D1, IC8A.D2, IC8A.D3, IC8A.POL
- new net N$39: IC6A.Q0, IC6A.Q1, IC6A.Q2, IC6A.Q3, IC7A.I0
- new net N$40: BUTTON_2.1
- new net N$41: BUTTON_3.2, R4.1
- new net N$42: C4.1, IC9A.D0, IC9A.D1, IC9A.D2, IC9A.D3, IC9A.POL, R4.2, R5.2
- new net N$43: IC10A.D0, IC10A.D1, IC10A.D2, IC10A.D3, IC10A.POL, IC9A.Q0, IC9A.Q1, IC9A.Q2, IC9A.Q3
- new net N$44: IC11A.I1, IC12A.Q0, IC12A.Q1, IC12A.Q2, IC12A.Q3
- new net N$45: IC10A.!Q0, IC10A.!Q1, IC10A.!Q2, IC10A.!Q3, IC12A.D0, IC12A.D1, IC12A.D2, IC12A.D3, IC12A.POL
- new net N$46: IC10A.Q0, IC10A.Q1, IC10A.Q2, IC10A.Q3, IC11A.I0
- new net N$47: BUTTON_3.1
- new net N$48: BUTTON_4.2, R6.1
- new net N$49: C2.1, IC1A.D0, IC1A.D1, IC1A.D2, IC1A.D3, IC1A.POL, R1.2, R17.2
- new net N$50: C5.1, IC13A.D0, IC13A.D1, IC13A.D2, IC13A.D3, IC13A.POL, R6.2, R7.2
- new net N$51: IC13A.Q0, IC13A.Q1, IC13A.Q2, IC13A.Q3, IC14A.D0, IC14A.D1, IC14A.D2, IC14A.D3, IC14A.POL
- new net N$52: IC15A.I1, IC16A.Q0, IC16A.Q1, IC16A.Q2, IC16A.Q3
- new net N$53: IC14A.!Q0, IC14A.!Q1, IC14A.!Q2, IC14A.!Q3, IC16A.D0, IC16A.D1, IC16A.D2, IC16A.D3, IC16A.POL
- new net N$54: IC14A.Q0, IC14A.Q1, IC14A.Q2, IC14A.Q3, IC15A.I0
- new net N$55: BUTTON_4.1
- new net N$56: BUTTON_5.2, R8.1
- new net N$57: C6.1, IC17A.D0, IC17A.D1, IC17A.D2, IC17A.D3, IC17A.POL, R8.2, R9.2
- new net N$58: IC17A.Q0, IC17A.Q1, IC17A.Q2, IC17A.Q3, IC18A.D0, IC18A.D1, IC18A.D2, IC18A.D3, IC18A.POL
- new net N$59: IC19A.I1, IC20A.Q0, IC20A.Q1, IC20A.Q2, IC20A.Q3
- new net N$60: IC18A.!Q0, IC18A.!Q1, IC18A.!Q2, IC18A.!Q3, IC20A.D0, IC20A.D1, IC20A.D2, IC20A.D3, IC20A.POL
- new net N$61: IC18A.Q0, IC18A.Q1, IC18A.Q2, IC18A.Q3, IC19A.I0
- new net N$62: BUTTON_5.1
- new net N$63: BUTTON_6.2, R10.1
- new net N$64: C7.1, IC21A.D0, IC21A.D1, IC21A.D2, IC21A.D3, IC21A.POL, R10.2, R11.2
- new net N$65: IC1A.Q0, IC1A.Q1, IC1A.Q2, IC1A.Q3, IC2A.D0, IC2A.D1, IC2A.D2, IC2A.D3, IC2A.POL
- new net N$66: IC21A.Q0, IC21A.Q1, IC21A.Q2, IC21A.Q3, IC22A.D0, IC22A.D1, IC22A.D2, IC22A.D3, IC22A.POL
- new net N$68: IC23A.I1, IC24A.Q0, IC24A.Q1, IC24A.Q2, IC24A.Q3
- new net N$69: IC3A.I1, IC4A.Q0, IC4A.Q1, IC4A.Q2, IC4A.Q3
- new net N$7: BUTTON_1.2, R1.1
- new net N$70: IC2A.!Q0, IC2A.!Q1, IC2A.!Q2, IC2A.!Q3, IC4A.D0, IC4A.D1, IC4A.D2, IC4A.D3, IC4A.POL
- new net N$71: IC22A.!Q0, IC22A.!Q1, IC22A.!Q2, IC22A.!Q3, IC24A.D0, IC24A.D1, IC24A.D2, IC24A.D3, IC24A.POL
- new net N$72: IC22A.Q0, IC22A.Q1, IC22A.Q2, IC22A.Q3, IC23A.I0
- new net N$73: BUTTON_6.1
- new net N$74: BUTTON_7.2, R12.1
- new net N$75: C8.1, IC25A.D0, IC25A.D1, IC25A.D2, IC25A.D3, IC25A.POL, R12.2, R13.2
- new net N$76: IC25A.Q0, IC25A.Q1, IC25A.Q2, IC25A.Q3, IC26A.D0, IC26A.D1, IC26A.D2, IC26A.D3, IC26A.POL
- new net N$77: IC2A.Q0, IC2A.Q1, IC2A.Q2, IC2A.Q3, IC3A.I0
- new net N$78: IC27A.I1, IC28A.Q0, IC28A.Q1, IC28A.Q2, IC28A.Q3
- new net N$79: IC26A.!Q0, IC26A.!Q1, IC26A.!Q2, IC26A.!Q3, IC28A.D0, IC28A.D1, IC28A.D2, IC28A.D3, IC28A.POL
- new net N$80: IC26A.Q0, IC26A.Q1, IC26A.Q2, IC26A.Q3, IC27A.I0
- new net N$81: BUTTON_7.1
- new net N$82: BUTTON_8.2, R14.1
- new net N$83: C9.1, IC29A.D0, IC29A.D1, IC29A.D2, IC29A.D3, IC29A.POL, R14.2, R15.2
- new net N$84: IC29A.Q0, IC29A.Q1, IC29A.Q2, IC29A.Q3, IC30A.D0, IC30A.D1, IC30A.D2, IC30A.D3, IC30A.POL
- new net N$85: IC31A.I1, IC32A.Q0, IC32A.Q1, IC32A.Q2, IC32A.Q3
- new net N$86: IC30A.!Q0, IC30A.!Q1, IC30A.!Q2, IC30A.!Q3, IC32A.D0, IC32A.D1, IC32A.D2, IC32A.D3, IC32A.POL
- new net N$87: IC30A.Q0, IC30A.Q1, IC30A.Q2, IC30A.Q3, IC31A.I0
- new net N$88: BUTTON_8.1
- new net N$89: BUTTON_9.2, R16.1
- new net N$90: C10.1, IC33A.D0, IC33A.D1, IC33A.D2, IC33A.D3, IC33A.POL, R16.2, R18.2
- new net N$91: IC33A.Q0, IC33A.Q1, IC33A.Q2, IC33A.Q3, IC34A.D0, IC34A.D1, IC34A.D2, IC34A.D3, IC34A.POL
- new net N$92: IC35A.I1, IC36A.Q0, IC36A.Q1, IC36A.Q2, IC36A.Q3
- new net N$93: IC34A.!Q0, IC34A.!Q1, IC34A.!Q2, IC34A.!Q3, IC36A.D0, IC36A.D1, IC36A.D2, IC36A.D3, IC36A.POL
- new net N$94: IC34A.Q0, IC34A.Q1, IC34A.Q2, IC34A.Q3, IC35A.I0
- new net N$95: BUTTON_9.1
- new net N$96: BUTTON_10.2, R19.1
- new net N$97: C11.1, IC37A.D0, IC37A.D1, IC37A.D2, IC37A.D3, IC37A.POL, R19.2, R20.2
- new net N$98: IC37A.Q0, IC37A.Q1, IC37A.Q2, IC37A.Q3, IC38A.D0, IC38A.D1, IC38A.D2, IC38A.D3, IC38A.POL
- new net N$99: IC39A.I1, IC40A.Q0, IC40A.Q1, IC40A.Q2, IC40A.Q3
- new net OUTPUT: IC11A.O, IC15A.O, IC19A.O, IC23A.O, IC27A.O, IC31A.O, IC35A.O, IC39A.O, IC3A.O, IC43A.O, IC47A.O, IC51A.O, IC55A.O, IC59A.O, IC63A.O, IC7A.O
- net GND: now also BUTTON_1.1, C10.2, C11.2, C12.2, C13.2, C14.2, C15.2, C16.2, C17.2, C2.2, C3.2, C4.2, C5.2, C6.2, C7.2, C8.2, C9.2, IC12A.!Q0, IC12A.!Q1, IC12A.!Q2, IC12A.!Q3, IC13A.!Q0, IC13A.!Q1, IC13A.!Q2, IC13A.!Q3, IC16A.!Q0, IC16A.!Q1, IC16A.!Q2, IC16A.!Q3, IC17A.!Q0, IC17A.!Q1, IC17A.!Q2, IC17A.!Q3, IC1A.!Q0, IC1A.!Q1, IC1A.!Q2, IC1A.!Q3, IC20A.!Q0, IC20A.!Q1, IC20A.!Q2, IC20A.!Q3, IC21A.!Q0, IC21A.!Q1, IC21A.!Q2, IC21A.!Q3, IC24A.!Q0, IC24A.!Q1, IC24A.!Q2, IC24A.!Q3, IC25A.!Q0, IC25A.!Q1, IC25A.!Q2, IC25A.!Q3, IC28A.!Q0, IC28A.!Q1, IC28A.!Q2, IC28A.!Q3, IC29A.!Q0, IC29A.!Q1, IC29A.!Q2, IC29A.!Q3, IC32A.!Q0, IC32A.!Q1, IC32A.!Q2, IC32A.!Q3, IC33A.!Q0, IC33A.!Q1, IC33A.!Q2, IC33A.!Q3, IC36A.!Q0, IC36A.!Q1, IC36A.!Q2, IC36A.!Q3, IC37A.!Q0, IC37A.!Q1, IC37A.!Q2, IC37A.!Q3, IC40A.!Q0, IC40A.!Q1, IC40A.!Q2, IC40A.!Q3, IC41A.!Q0, IC41A.!Q1, IC41A.!Q2, IC41A.!Q3, IC44A.!Q0, IC44A.!Q1, IC44A.!Q2, IC44A.!Q3, IC45A.!Q0, IC45A.!Q1, IC45A.!Q2, IC45A.!Q3, IC48A.!Q0, IC48A.!Q1, IC48A.!Q2, IC48A.!Q3, IC49A.!Q0, IC49A.!Q1, IC49A.!Q2, IC49A.!Q3, IC4A.!Q0, IC4A.!Q1, IC4A.!Q2, IC4A.!Q3, IC52A.!Q0, IC52A.!Q1, IC52A.!Q2, IC52A.!Q3, IC53A.!Q0, IC53A.!Q1, IC53A.!Q2, IC53A.!Q3, IC56A.!Q0, IC56A.!Q1, IC56A.!Q2, IC56A.!Q3, IC57A.!Q0, IC57A.!Q1, IC57A.!Q2, IC57A.!Q3, IC5A.!Q0, IC5A.!Q1, IC5A.!Q2, IC5A.!Q3, IC60A.!Q0, IC60A.!Q1, IC60A.!Q2, IC60A.!Q3, IC61A.!Q0, IC61A.!Q1, IC61A.!Q2, IC61A.!Q3, IC64A.!Q0, IC64A.!Q1, IC64A.!Q2, IC64A.!Q3, IC8A.!Q0, IC8A.!Q1, IC8A.!Q2, IC8A.!Q3, IC9A.!Q0, IC9A.!Q1, IC9A.!Q2, IC9A.!Q3, R11.1, R13.1, R15.1, R17.1, R18.1, R20.1, R22.1, R24.1, R26.1, R28.1, R3.1, R30.1, R32.1, R5.1, R7.1, R9.1
Other:
- note added: "Delays"
