File: MainBoard/Instruments.sch (EAGLE design)
At the start: 9 parts

Commit message: Completed schematics
Peliminary files of completed schematics (Hopefully with proper connections this time...)
Parts:
- renumbered JP1 to KICK_DRUM, JP2 to HI_TOM, JP3 to LOW_TOM, JP4 to SNARE_DRUM, JP5 to CRASH, JP6 to HI-HAT, JP7 to CLOSED_HI-HAT, JP8 to COWBELL, MIXER1 to MIXER
