File: Kick Drum/EAGLE/Analog Drum/Analog Drum.sch (EAGLE design)
At the start: 57 parts, among them IC1 LM741P, IC2 LM741P, IC3 LM741P, IC4 LM741P, IC5 LM741P, Q1 2N3906, Q2 2N3906, T1 2N3904, T2 2N3904, T3 2N3904, T4 2N3904

Commit message: work on schematic
Parts:
- added R29, R30, R31, R32, R33: (no value), resistor:R-US_0207/10
Connections:
- new net N$23: IC4.-IN, R29.2
- new net N$27: IC4.+IN, R30.2
- new net N$28: IC4.OUT, R31.2
- new net N$29: IC5.-IN, R31.1, R32.2
- new net N$31: IC5.OUT, R32.1, R33.2
- new net N$32: R33.1
- net +12V: now also IC2.V+, IC3.V+, IC4.V+, IC5.V+
- net -12V: now also IC2.V-, IC3.V-, IC4.V-, IC5.V-
- net 0V: now also R30.1
- net RES_FTR_OUT: now also R29.1
Other:
- moved on the sheet: IC4, IC5, R24, R27, R28
