File: Kick Drum/EAGLE/Analog Drum.brd (EAGLE design)
At the start: 100 x 50 mm, 78 parts, among them IC1 LM741P, IC2 LM741P, IC3 LM741P, IC4 LM741P, IC5 LM741P, Q1 2N3906, Q2 2N3906, T2 2N3904, T3 2N3904, T4 2N3904

Commit message: work on pcb.
-laying out components
Parts:
- moved R37 175.4 mm to (86.0, 23.0), turned to 270 degrees
- moved R19 175.2 mm to (96.3, 11.8), turned to 270 degrees
- moved C9 165.5 mm to (95.0, 22.0), turned to 180 degrees
- moved D3 157.5 mm to (89.0, 18.0)
- moved D4 156.0 mm to (70.0, 14.0), turned to 90 degrees
- moved R18 155.1 mm to (87.0, 10.0), turned to 180 degrees
- moved C10 153.5 mm to (74.0, 12.0), turned to 90 degrees
- moved C8 143.4 mm to (79.0, 12.0), turned to 90 degrees
- moved D2 140.5 mm to (87.0, 14.0)
- moved T4 137.5 mm to (73.0, 24.0)
- moved IC3 123.9 mm to (79.0, 38.0), turned to 270 degrees
- moved R24 119.0 mm to (66.0, 28.0), turned to 180 degrees
- moved R21 105.7 mm to (73.0, 20.6), turned to 180 degrees
- moved IC5 104.3 mm to (34.0, 38.0), turned to 270 degrees
- moved C25 103.4 mm to (33.0, 31.0), turned to 180 degrees
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Connections:
- net POT5: now also R2.3; no longer R2.1
