File: VU meter/VU meter schematic.brd (EAGLE design)
At the start: 35 x 40 mm, 5 parts

Commit message: u don ducked
Parts:
- added R1: 630, resistor:0207/10
- added R6, R9: 10k, resistor:0207/10
- added R7: 470, resistor:0207/10
- added R8: 100, resistor:0207/10
- moved D2 12.0 mm to (16.9, 17.8)
- moved C1 11.4 mm to (5.76, 17.8)
- moved D1 6.40 mm to (17.7, 27.7)
Connections:
- new net N$5: R1.2, R9.2
- net N$1: now also R6.1
- net N$2: now also R6.2, R7.1, R8.1, R9.1
- net N$3: now also R1.1
- net N$6: now also R8.2
- net N$8: now also R7.2
Routing:
- net N$3: track 31.9 -> 0.17 mm
Changed lines of the file:
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@@
 <layers>
 <layer number="1" name="Top" color="4" fill="1" visible="yes" active="yes"/>
+<layer number="2" name="Route2" color="1" fill="3" visible="no" active="no"/>
+<layer number="3" name="Route3" color="4" fill="3" visible="no" active="no"/>
+<layer number="4" name="Route4" color="1" fill="4" visible="no" active="no"/>
+<layer number="5" name="Route5" color="4" fill="4" visible="no" active="no"/>
+<layer number="6" name="Route6" color="1" fill="8" visible="no" active="no"/>
+<layer number="7" name="Route7" color="4" fill="8" visible="no" active="no"/>
+<layer number="8" name="Route8" color="1" fill="2" visible="no" active="no"/>
+<layer number="9" name="Route9" color="4" fill="2" visible="no" active="no"/>
+<layer number="10" name="Route10" color="1" fill="7" visible="no" active="no"/>
+<layer number="11" name="Route11" color="4" fill="7" visible="no" active="no"/>
+<layer number="12" name="Route12" color="1" fill="5" visible="no" active="no"/>
+<layer number="13" name="Route13" color="4" fill="5" visible="no" active="no"/>
+<layer number="14" name="Route14" color="1" fill="6" visible="no" active="no"/>
+<layer number="15" name="Route15" color="4" fill="6" visible="no" active="no"/>
 <layer number="16" name="Bottom" color="1" fill="1" visible="yes" active="yes"/>
 <layer number="17" name="Pads" color="2" fill="1" visible="yes" active="yes"/>
@@
 <wire x1="35" y1="40" x2="0" y2="40" width="0" layer="20"/>
 <wire x1="0" y1="40" x2="0" y2="0" width="0" layer="20"/>
-<text x="8" y="20" size="1.778" layer="21">VU meter circuit</text>
+<text x="9" y="13" size="1.778" layer="21">VU meter circuit</text>
 </plain>
 <attributes>
@@
 </autorouter>
 <elements>
-<element name="C1" library="capacitor-wima" library_urn="urn:adsk.eagle:library:116" package="C2.5-3" package3d_urn="urn:adsk.eagle:package:5436/1" value="4u7" x="16.76" y="14.81" smashed="yes">
-<attribute name="NAME" x="17.109" y="17.588" size="1.27" layer="25" ratio="10"/>
-<attribute name="VALUE" x="15.109" y="11.762" size="1.27" layer="27" ratio="10"/>
-</element>
-<element name="D1" library="diode" library_urn="urn:adsk.eagle:library:210" package="DO35-10" package3d_urn="urn:adsk.eagle:package:43344/2" value="BAT42" x="13.68" y="32.67" smashed="yes">
-<attribute name="NAME" x="11.521" y="33.94" size="1.27" layer="25" ratio="10"/>
-<attribute name="VALUE" x="11.521" y="30.003" size="1.27" layer="27" ratio="10"/>
-</element>
-<element name="D2" library="diode" library_urn="urn:adsk.eagle:library:210" package="DO41-10" package3d_urn="urn:adsk.eagle:package:43336/1" value="1N4004" x="16.87" y="5.81" smashed="yes">
-<attribute name="NAME" x="14.838" y="7.461" size="1.27" layer="25" ratio="10"/>
-<attribute name="VALUE" x="14.838" y="3.016" size="1.27" layer="27" ratio="10"/>
+<element name="C1" library="capacitor-wima" library_urn="urn:adsk.eagle:library:116" package="C2.5-3" package3d_urn="urn:adsk.eagle:package:5436/1" value="4u7" x="5.76" y="17.81" smashed="yes">
+<attribute name="NAME" x="4.109" y="19.588" size="1.27" layer="25" ratio="10"/>
+<attribute name="VALUE" x="4.109" y="14.762" size="1.27" layer="27" ratio="10"/>
+</element>
+<element name="D1" library="diode" library_urn="urn:adsk.eagle:library:210" package="DO35-10" package3d_urn="urn:adsk.eagle:package:43344/2" value="BAT42" x="17.68" y="27.67" smashed="yes">
+<attribute name="NAME" x="15.521" y="28.94" size="1.27" layer="25" ratio="10"/>
+<attribute name="VALUE" x="15.521" y="25.003" size="1.27" layer="27" ratio="10"/>
+</element>
+<element name="D2" library="diode" library_urn="urn:adsk.eagle:library:210" package="DO41-10" package3d_urn="urn:adsk.eagle:package:43336/1" value="1N4004" x="16.87" y="17.81" smashed="yes">
+<attribute name="NAME" x="14.838" y="19.461" size="1.27" layer="25" ratio="10"/>
+<attribute name="VALUE" x="14.838" y="15.016" size="1.27" layer="27" ratio="10"/>
 </element>
 <element name="D3" library="diode" library_urn="urn:adsk.eagle:library:210" package="DO41-10" package3d_urn="urn:adsk.eagle:package:43336/1" value="1N4004" x="25.93" y="24.05" smashed="yes">
@@
 <attribute name="NAME" x="6.918" y="25.701" size="1.27" layer="25" ratio="10"/>
 <attribute name="VALUE" x="6.918" y="21.256" size="1.27" layer="27" ratio="10"/>
+</element>
+<element name="R6" library="resistor" library_urn="urn:adsk.eagle:library:348" package="0207/10" package3d_urn="urn:adsk.eagle:package:25939/1" value="10k" x="6" y="-4" smashed="yes">
+<attribute name="NAME" x="2.952" y="-2.476" size="1.27" layer="25" ratio="10"/>
+<attribute name="VALUE" x="3.7394" y="-4.635" size="1.27" layer="27" ratio="10"/>
+</element>
+<element name="R7" library="resistor" library_urn="urn:adsk.eagle:library:348" package="0207/10" package3d_urn="urn:adsk.eagle:package:25939/1" value="470" x="6" y="-9" smashed="yes">
+<attribute name="NAME" x="2.952" y="-7.476" size="1.27" layer="25" ratio="10"/>
+<attribute name="VALUE" x="3.7394" y="-9.635" size="1.27" layer="27" ratio="10"/>
+</element>
+<element name="R8" library="resistor" library_urn="urn:adsk.eagle:library:348" package="0207/10" package3d_urn="urn:adsk.eagle:package:25939/1" value="100" x="6" y="-14" smashed="yes">
+<attribute name="NAME" x="2.952" y="-12.476" size="1.27" layer="25" ratio="10"/>
+<attribute name="VALUE" x="3.7394" y="-14.635" size="1.27" layer="27" ratio="10"/>
+</element>
+<element name="R9" library="resistor" library_urn="urn:adsk.eagle:library:348" package="0207/10" package3d_urn="urn:adsk.eagle:package:25939/1" value="10k" x="6" y="-19" smashed="yes">
+<attribute name="NAME" x="2.952" y="-17.476" size="1.27" layer="25" ratio="10"/>
+<attribute name="VALUE" x="3.7394" y="-19.635" size="1.27" layer="27" ratio="10"/>
+</element>
+<element name="R1" library="resistor" library_urn="urn:adsk.eagle:library:348" package="0207/10" package3d_urn="urn:adsk.eagle:package:25939/1" value="630" x="6" y="-24" smashed="yes">
+<attribute name="NAME" x="2.952" y="-22.476" size="1.27" layer="25" ratio="10"/>
+<attribute name="VALUE" x="3.7394" y="-24.635" size="1.27" layer="27" ratio="10"/>
 </element>
 </elements>
@@
 <signal name="N$1">
 <contactref element="D1" pad="C"/>
+<contactref element="R6" pad="1"/>
+<wire x1="0.92" y1="-4" x2="12.6" y2="27.67" width="0" layer="19" extent="1-1"/>
 </signal>
 <signal name="N$2">
 <contactref element="C1" pad="1"/>
+<contactref element="R6" pad="2"/>
+<contactref element="R7" pad="1"/>
+<contactref element="R8" pad="1"/>
+<contactref element="R9" pad="1"/>
+<wire x1="11.08" y1="-4" x2="4.49" y2="17.81" width="0" layer="19" extent="1-1"/>
+<wire x1="0.92" y1="-9" x2="11.08" y2="-4" width="0" layer="19" extent="1-1"/>
+<wire x1="0.92" y1="-14" x2="0.92" y2="-9" width="0" layer="19" extent="1-1"/>
+<wire x1="0.92" y1="-19" x2="0.92" y2="-14" width="0" layer="19" extent="1-1"/>
 </signal>
 <signal name="N$3">
@@
 <contactref element="D2" pad="C"/>
 <contactref element="D4" pad="C"/>
-<wire x1="18" y1="12" x2="18" y2="14.75" width="0.3048" layer="1"/>
-<wire x1="11.875" y1="5.875" x2="18" y2="12" width="0.3048" layer="1"/>
-<wire x1="18" y1="14.75" x2="18.03" y2="14.81" width="0.3048" layer="1"/>
-<wire x1="11.875" y1="5.875" x2="11.79" y2="5.81" width="0.3048" layer="1"/>
-<wire x1="18.03" y1="14.81" x2="15.03" y2="17.81" width="0.3048" layer="1"/>
-<wire x1="15.03" y1="17.81" x2="6.065" y2="17.81" width="0.3048" layer="1"/>
-<wire x1="6.065" y1="17.81" x2="3.87" y2="20.005" width="0.3048" layer="1"/>
-<wire x1="3.87" y1="24.05" x2="3.87" y2="20.005" width="0.3048" layer="1"/>
+<wire x1="7" y1="17.75" x2="7.03" y2="17.81" width="0.3048" layer="1"/>
+<wire x1="11.875" y1="17.875" x2="11.79" y2="17.81" width="0.3048" layer="1"/>
+<contactref element="R1" pad="1"/>
+<wire x1="11.875" y1="17.875" x2="7" y2="17.75" width="0" layer="19" extent="1-1"/>
+<wire x1="3.87" y1="24.05" x2="7.03" y2="17.81" width="0" layer="19" extent="1-1"/>
+<wire x1="0.92" y1="-24" x2="11.79" y2="17.81" width="0" layer="19" extent="1-1"/>
 </signal>
 <signal name="N$4">
@@
 <signal name="N$6">
 <contactref element="D3" pad="A"/>
+<contactref element="R8" pad="2"/>
+<wire x1="11.08" y1="-14" x2="31.01" y2="24.05" width="0" layer="19" extent="1-1"/>
 </signal>
 <signal name="N$7">
@@
 <signal name="N$8">
 <contactref element="D2" pad="A"/>
+<contactref element="R7" pad="2"/>
+<wire x1="11.08" y1="-9" x2="21.95" y2="17.81" width="0" layer="19" extent="1-1"/>
 </signal>
 <signal name="GND">
@@
 </polygon>
 </signal>
+<signal name="N$5">
+<contactref element="R1" pad="2"/>
+<contactref element="R9" pad="2"/>
+<wire x1="11.08" y1="-19" x2="11.08" y2="-24" width="0" layer="19" extent="1-1"/>
+</signal>
 </signals>
