File: VU meter/VU meter schematic.sch (EAGLE design)
At the start: 10 parts

Commit message: u don ducked
Parts:
- removed R2: 470, ngspice-simulation:R
- removed R3: 100, ngspice-simulation:R
- removed R4: 10k, ngspice-simulation:R
- removed R5: 630, ngspice-simulation:R
- added R6, R9: 10k, resistor:R-US_0207/10
- added R7: 470, resistor:R-US_0207/10
- added R8: 100, resistor:R-US_0207/10
- R1: value 10k -> 630; device ngspice-simulation:R -> resistor:R-US_0207/10
Connections:
- net N$1: now also R6.1; no longer R1.1
- net N$2: now also R6.2, R7.1, R8.1, R9.1; no longer R1.2, R2.2, R3.2, R4.2
- net N$3: now also R1.1; no longer R5.2
- net N$5: now also R1.2, R9.2; no longer R4.1, R5.1
- net N$6: now also R8.2; no longer R3.1
- net N$8: now also R7.2; no longer R2.1
Changed lines of the file:
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@@
 <layers>
 <layer number="1" name="Top" color="4" fill="1" visible="no" active="no"/>
+<layer number="2" name="Route2" color="1" fill="3" visible="no" active="no"/>
+<layer number="3" name="Route3" color="4" fill="3" visible="no" active="no"/>
+<layer number="4" name="Route4" color="1" fill="4" visible="no" active="no"/>
+<layer number="5" name="Route5" color="4" fill="4" visible="no" active="no"/>
+<layer number="6" name="Route6" color="1" fill="8" visible="no" active="no"/>
+<layer number="7" name="Route7" color="4" fill="8" visible="no" active="no"/>
+<layer number="8" name="Route8" color="1" fill="2" visible="no" active="no"/>
+<layer number="9" name="Route9" color="4" fill="2" visible="no" active="no"/>
+<layer number="10" name="Route10" color="1" fill="7" visible="no" active="no"/>
+<layer number="11" name="Route11" color="4" fill="7" visible="no" active="no"/>
+<layer number="12" name="Route12" color="1" fill="5" visible="no" active="no"/>
+<layer number="13" name="Route13" color="4" fill="5" visible="no" active="no"/>
+<layer number="14" name="Route14" color="1" fill="6" visible="no" active="no"/>
+<layer number="15" name="Route15" color="4" fill="6" visible="no" active="no"/>
 <layer number="16" name="Bottom" color="1" fill="1" visible="no" active="no"/>
 <layer number="17" name="Pads" color="2" fill="1" visible="no" active="no"/>
@@
 <part name="D1" library="diode" library_urn="urn:adsk.eagle:library:210" deviceset="BAT42" device="" package3d_urn="urn:adsk.eagle:package:43344/2"/>
 <part name="C1" library="capacitor-wima" library_urn="urn:adsk.eagle:library:116" deviceset="C" device="2,5-3" package3d_urn="urn:adsk.eagle:package:5436/1" value="4u7"/>
-<part name="R1" library="ngspice-simulation" library_urn="urn:adsk.eagle:library:527439" deviceset="R" device="" value="10k"/>
-<part name="R2" library="ngspice-simulation" library_urn="urn:adsk.eagle:library:527439" deviceset="R" device="" value="470"/>
-<part name="R3" library="ngspice-simulation" library_urn="urn:adsk.eagle:library:527439" deviceset="R" device="" value="100"/>
-<part name="R4" library="ngspice-simulation" library_urn="urn:adsk.eagle:library:527439" deviceset="R" device="" value="10k"/>
 <part name="D2" library="diode" library_urn="urn:adsk.eagle:library:210" deviceset="1N4004" device="" package3d_urn="urn:adsk.eagle:package:43336/1"/>
 <part name="D3" library="diode" library_urn="urn:adsk.eagle:library:210" deviceset="1N4004" device="" package3d_urn="urn:adsk.eagle:package:43336/1"/>
 <part name="D4" library="diode" library_urn="urn:adsk.eagle:library:210" deviceset="1N4004" device="" package3d_urn="urn:adsk.eagle:package:43336/1"/>
-<part name="R5" library="ngspice-simulation" library_urn="urn:adsk.eagle:library:527439" deviceset="R" device="" value="630"/>
+<part name="R6" library="resistor" library_urn="urn:adsk.eagle:library:348" deviceset="R-US_" device="0207/10" package3d_urn="urn:adsk.eagle:package:25939/1" value="10k"/>
+<part name="R7" library="resistor" library_urn="urn:adsk.eagle:library:348" deviceset="R-US_" device="0207/10" package3d_urn="urn:adsk.eagle:package:25939/1" value="470"/>
+<part name="R8" library="resistor" library_urn="urn:adsk.eagle:library:348" deviceset="R-US_" device="0207/10" package3d_urn="urn:adsk.eagle:package:25939/1" value="100"/>
+<part name="R9" library="resistor" library_urn="urn:adsk.eagle:library:348" deviceset="R-US_" device="0207/10" package3d_urn="urn:adsk.eagle:package:25939/1" value="10k"/>
+<part name="R1" library="resistor" library_urn="urn:adsk.eagle:library:348" deviceset="R-US_" device="0207/10" package3d_urn="urn:adsk.eagle:package:25939/1" value="630"/>
 </parts>
 <sheets>
@@
 <attribute name="VALUE" x="54.864" y="56.261" size="1.778" layer="96" rot="R90"/>
 </instance>
-<instance part="R1" gate="G$1" x="43.18" y="73.66" smashed="yes">
-<attribute name="NAME" x="40.64" y="76.2" size="1.778" layer="95"/>
-<attribute name="VALUE" x="40.64" y="69.85" size="1.778" layer="96"/>
-</instance>
-<instance part="R2" gate="G$1" x="66.04" y="66.04" smashed="yes" rot="R90">
-<attribute name="NAME" x="63.5" y="63.5" size="1.778" layer="95" rot="R90"/>
-<attribute name="VALUE" x="69.85" y="63.5" size="1.778" layer="96" rot="R90"/>
-</instance>
-<instance part="R3" gate="G$1" x="83.82" y="66.04" smashed="yes" rot="R90">
-<attribute name="NAME" x="81.28" y="63.5" size="1.778" layer="95" rot="R90"/>
-<attribute name="VALUE" x="87.63" y="63.5" size="1.778" layer="96" rot="R90"/>
-</instance>
-<instance part="R4" gate="G$1" x="93.98" y="73.66" smashed="yes" rot="R180">
-<attribute name="NAME" x="93.98" y="78.74" size="1.778" layer="95" rot="R180"/>
-<attribute name="VALUE" x="96.52" y="72.39" size="1.778" layer="96" rot="R180"/>
-</instance>
 <instance part="D2" gate="1" x="66.04" y="55.88" smashed="yes" rot="R270">
 <attribute name="NAME" x="61.4426" y="55.88" size="1.778" layer="95" rot="R270"/>
@@
 <attribute name="VALUE" x="86.5886" y="48.26" size="1.778" layer="96" rot="R270"/>
 </instance>
-<instance part="R5" gate="G$1" x="104.14" y="53.34" smashed="yes" rot="R270">
-<attribute name="NAME" x="106.68" y="55.88" size="1.778" layer="95" rot="R270"/>
-<attribute name="VALUE" x="100.33" y="55.88" size="1.778" layer="96" rot="R270"/>
+<instance part="R6" gate="G$1" x="43.18" y="73.66" smashed="yes">
+<attribute name="NAME" x="39.37" y="75.1586" size="1.778" layer="95"/>
+<attribute name="VALUE" x="39.37" y="70.358" size="1.778" layer="96"/>
+</instance>
+<instance part="R7" gate="G$1" x="66.04" y="66.04" smashed="yes" rot="R270">
+<attribute name="NAME" x="67.5386" y="69.85" size="1.778" layer="95" rot="R270"/>
+<attribute name="VALUE" x="62.738" y="69.85" size="1.778" layer="96" rot="R270"/>
+</instance>
+<instance part="R8" gate="G$1" x="83.82" y="66.04" smashed="yes" rot="R270">
+<attribute name="NAME" x="85.3186" y="69.85" size="1.778" layer="95" rot="R270"/>
+<attribute name="VALUE" x="80.518" y="69.85" size="1.778" layer="96" rot="R270"/>
+</instance>
+<instance part="R9" gate="G$1" x="93.98" y="73.66" smashed="yes">
+<attribute name="NAME" x="90.17" y="75.1586" size="1.778" layer="95"/>
+<attribute name="VALUE" x="90.17" y="70.358" size="1.778" layer="96"/>
+</instance>
+<instance part="R1" gate="G$1" x="104.14" y="53.34" smashed="yes" rot="R90">
+<attribute name="NAME" x="102.6414" y="49.53" size="1.778" layer="95" rot="R90"/>
+<attribute name="VALUE" x="107.442" y="49.53" size="1.778" layer="96" rot="R90"/>
 </instance>
 </instances>
@@
 <pinref part="D1" gate="1" pin="C"/>
 <wire x1="30.48" y1="73.66" x2="38.1" y2="73.66" width="0.1524" layer="91"/>
-<pinref part="R1" gate="G$1" pin="1"/>
+<pinref part="R6" gate="G$1" pin="1"/>
 </segment>
 </net>
@@
 <wire x1="50.8" y1="73.66" x2="50.8" y2="60.96" width="0.1524" layer="91"/>
 <pinref part="C1" gate="G$1" pin="1"/>
-<pinref part="R1" gate="G$1" pin="2"/>
 <wire x1="50.8" y1="73.66" x2="66.04" y2="73.66" width="0.1524" layer="91"/>
 <junction x="50.8" y="73.66"/>
-<pinref part="R2" gate="G$1" pin="2"/>
 <wire x1="66.04" y1="73.66" x2="66.04" y2="71.12" width="0.1524" layer="91"/>
-<pinref part="R3" gate="G$1" pin="2"/>
 <wire x1="66.04" y1="73.66" x2="83.82" y2="73.66" width="0.1524" layer="91"/>
 <wire x1="83.82" y1="73.66" x2="83.82" y2="71.12" width="0.1524" layer="91"/>
 <junction x="66.04" y="73.66"/>
-<pinref part="R4" gate="G$1" pin="2"/>
 <wire x1="88.9" y1="73.66" x2="83.82" y2="73.66" width="0.1524" layer="91"/>
 <junction x="83.82" y="73.66"/>
-<wire x1="83.82" y1="73.66" x2="83.82" y2="78.74" width="0.1524" layer="91"/>
-<wire x1="83.82" y1="78.74" x2="93.98" y2="78.74" width="0.1524" layer="91"/>
-<wire x1="93.98" y1="78.74" x2="93.98" y2="73.66" width="0.1524" layer="91"/>
+<pinref part="R6" gate="G$1" pin="2"/>
+<pinref part="R7" gate="G$1" pin="1"/>
+<pinref part="R8" gate="G$1" pin="1"/>
+<pinref part="R9" gate="G$1" pin="1"/>
 </segment>
 </net>
@@
 <wire x1="83.82" y1="35.56" x2="66.04" y2="35.56" width="0.1524" layer="91"/>
 <junction x="66.04" y="35.56"/>
-<pinref part="R5" gate="G$1" pin="2"/>
 <wire x1="83.82" y1="35.56" x2="104.14" y2="35.56" width="0.1524" layer="91"/>
 <wire x1="104.14" y1="35.56" x2="104.14" y2="48.26" width="0.1524" layer="91"/>
 <junction x="83.82" y="35.56"/>
+<pinref part="R1" gate="G$1" pin="1"/>
 </segment>
 </net>
@@
 <net name="N$6" class="0">
 <segment>
-<pinref part="R3" gate="G$1" pin="1"/>
 <pinref part="D3" gate="1" pin="A"/>
 <wire x1="83.82" y1="60.96" x2="83.82" y2="58.42" width="0.1524" layer="91"/>
+<pinref part="R8" gate="G$1" pin="2"/>
 </segment>
 </net>
@@
 <net name="N$5" class="0">
 <segment>
-<pinref part="R4" gate="G$1" pin="1"/>
-<pinref part="R5" gate="G$1" pin="1"/>
 <wire x1="99.06" y1="73.66" x2="104.14" y2="73.66" width="0.1524" layer="91"/>
 <wire x1="104.14" y1="73.66" x2="104.14" y2="58.42" width="0.1524" layer="91"/>
+<pinref part="R1" gate="G$1" pin="2"/>
+<pinref part="R9" gate="G$1" pin="2"/>
 </segment>
 </net>
 <net name="N$8" class="0">
 <segment>
-<pinref part="R2" gate="G$1" pin="1"/>
 <pinref part="D2" gate="1" pin="A"/>
 <wire x1="66.04" y1="60.96" x2="66.04" y2="58.42" width="0.1524" layer="91"/>
+<pinref part="R7" gate="G$1" pin="2"/>
 </segment>
 </net>
@@
 packages will not be understood (or retained) with this version.
 </note>
-<note version="8.4" severity="warning">
-Since Version 8.4, EAGLE supports properties for SPICE simulation.
-Probes in schematics and SPICE mapping objects found in parts and library devices
-will not be understood with this version. Update EAGLE to the latest version
-for full support of SPICE simulation.
-</note>
 </compatibility>
