File: Mixer/Eagle Files/Mixer.sch (EAGLE design)
At the start: 45 parts, among them CON1 1-770875-01-770875-0_VERTICAL, IC1 LM741P, IC2 LM741P, T1 2N3904

Commit message: Implemented changes from design review meeting.
Parts:
- added C16, C17: 100uF, rcl:CPOL-USE5-8.5
- added C18, C19: 1u, resistor:C-EU050-024X044
- added R22: 50, rcl:R-US_0207/7
- added R23: PV36W101C01B00, Capstone:PV36W101C01B00
Connections:
- new net N$13: R22.1, R23.2
- net +12V: now also C16.+, C18.2, CON1.1; no longer CON1.4
- net +5V: now also CON1.3; no longer CON1.6
- net -12V: now also C17.-, C19.1, CON1.2; no longer CON1.5
- net GND: now also C16.-, C17.+, C18.1, C19.2, CON1.4, CON1.5, R23.3; no longer CON1.1, CON1.2, CON1.3
- net N$3: now also R22.2
Other:
- moved on the sheet: C10, C7, C8, C9, CON1, D3, D4, D5, D6, IC2, R20, R21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
