File: Analog Drums/EAGLE/Analog Drum.brd (EAGLE design)
At the start: 100 x 50 mm, 79 parts, among them IC1 LM741P, IC2 LM741P, IC3 LM741P, IC4 LM741P, IC5 LM741P, Q1 2N3906, Q2 2N3906, T2 2N3904, T3 2N3904, T4 2N3904

Commit message: cleanup
Routing:
- net N$14: track 8.52 -> 22.5 mm
- net N$5: track 0.00 -> 9.78 mm
Changed lines of the file:
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@@
 <wire x1="81.46" y1="6" x2="83.365" y2="7.905" width="0.254" layer="1"/>
 <contactref element="R38" pad="2"/>
-<wire x1="94.6" y1="3.92" x2="79" y2="6.27" width="0" layer="19" extent="1-1"/>
+<wire x1="94.6" y1="3.92" x2="93.92" y2="4.6" width="0.254" layer="16"/>
+<wire x1="82.86" y1="4.6" x2="81.46" y2="6" width="0.254" layer="16"/>
+<wire x1="93.92" y1="4.6" x2="82.86" y2="4.6" width="0.254" layer="16"/>
 </signal>
 <signal name="N$15">
@@
 <contactref element="Q2" pad="2"/>
 <contactref element="R38" pad="1"/>
-<wire x1="94.6" y1="14.08" x2="90" y2="7.905" width="0" layer="19" extent="1-1"/>
+<wire x1="94.6" y1="14.08" x2="94.6" y2="9.6" width="0.254" layer="16"/>
+<wire x1="92.905" y1="7.905" x2="90" y2="7.905" width="0.254" layer="16"/>
+<wire x1="94.6" y1="9.6" x2="92.905" y2="7.905" width="0.254" layer="16"/>
 </signal>
 </signals>
