File: PATA Breakout/PATA Breakout.brd (EAGLE design)
At the start: 60 x 20 mm, 5 parts

Commit message: cleanup
Parts:
- moved JP1 5.00 mm to (26.0, 15.0)
- moved SV1 5.00 mm to (26.0, 8.00)
- moved SV2 5.00 mm to (26.0, 22.0)
- moved SV3 5.00 mm to (56.9, 14.9)
- moved SV6 5.00 mm to (53.6, 14.9)
Other:
- board size 60 x 20 mm -> 60 x 30 mm
- board text added: "March 7 / 2019"
- board text added: "PATA Breakout Koltin Kosik-Harvey"
