File: Hi Hat/PCB/Hi-Hat.brd (EAGLE design)
At the start: 100 x 50 mm, 150 parts, among them IC1 LM741P, IC2 LM741P, IC3 LM741P, IC4 LM741P, IC5 LM741P, IC6 LM741P, IC7 LM741P, Q1 2N3904, Q10 2N2222A, Q11 2N2222A, Q12 2N2222A, Q13 2N2222A, Q14 2N2222A, Q2 2N3904, Q3 2N2222A, Q4 2N2222A, Q6 2N3904, Q7 2N2222A, Q8 2N2222A, Q9 2N2222A

Commit message: Completed most of hi-hat schematic
Parts:
- removed C10, C11, C12, C21, C22, C23, C24, C26, C28, C29, C35, C36, C9: 0.1uF, resistor:C050-024X044
- removed C19, C20: 0.33uF, resistor:C050-024X044
- removed C25, C27: 33nF, resistor:C050-024X044
- removed C30, C32: 2.2u, resistor:C050-024X044
- removed C31: 1u, resistor:C050-024X044
- removed C33: 10uF, rcl:E2,5-6
- removed C4: 1nF, resistor:C050-024X044
- removed D1, D2: 200mA/100V/1V, SparkFun-DiscreteSemi:DIODE-1N4148
- removed IC2, IC3, IC4, IC5, IC6: LM741P, linear:DIL08
- removed J1, J2: (no value), SparkFun-Connectors:2X3-NS
- removed J3, J4: (no value), SparkFun-Connectors:1X02_NO_SILK
- removed Q3, Q4: 2N2222A, SparkFun-DiscreteSemi:TO-92
- removed Q5: (no value), Capstone:TO-92
- removed Q6: 2N3904, transistor:TO92
- removed R1, R5: 15k, resistor:0207/10
- removed R10, R15, R17, R18, R21, R22, R28, R30, R35, R36, R41, R42, R44: 10k, resistor:0207/10
- removed R11, R6: 2k, resistor:0207/10
- removed R19, R20: 470k, resistor:0207/10
- removed R23: 100, resistor:0207/10
- removed R25: 51k, resistor:0207/10
- removed R26, R45: 47k, resistor:0207/10
- removed R27: 100k, resistor:0207/10
- removed R29, R32, R38: 1k, resistor:0207/10
- removed R31: 1meg, resistor:0207/10
- removed R43: 220, resistor:0207/10
- removed R7: 4.7k, resistor:0207/10
- removed TRIM1: 20 OHM, rcl:RTRIM64W
- removed TRIM2, TRIM3, TRIM4, TRIM5, TRIM6: 10k, rcl:RTRIM64W
- added C50: 0.47uF, resistor:C050-024X044
- added C51, C52: 0.1uF, resistor:C050-024X044
- added C53: 22nF, resistor:C050-024X044
- added C54, C56: 2.2u, resistor:C050-024X044
- added C55: 1u, resistor:C050-024X044
- added C57: 10uF, rcl:E2,5-6
- added C58: 1.5nF, resistor:C050-024X044
- added C59, C60: 1nF, resistor:C050-024X044
- added D3: 200mA/100V/1V, SparkFun-DiscreteSemi:DIODE-1N4148
- added IC8: LM741P, linear:DIL08
- added Q15: 2N2222A, SparkFun-DiscreteSemi:TO-92
- added Q16: (no value), Capstone:TO-92
- added Q17, Q18: 2N3904, transistor:TO92
- added R64, R68, R69, R70, R71, R75, R76, R77, R78: 10k, resistor:0207/10
- added R65, R83: 22k, resistor:0207/10
- added R66: 470k, resistor:0207/10
- added R67, R73, R80: 47k, resistor:0207/10
- added R72: 100, resistor:0207/10
- added R74: 18k, resistor:0207/10
- added R79: 220, resistor:0207/10
- added R81: 2.7k, resistor:0207/10
- added R82: 68k, resistor:0207/10
- added TRIM11: 10k, rcl:RTRIM64W
- added TRIM12: 20 OHM, rcl:RTRIM64W
- C2: value 1nF -> 0.1uF
- moved C2 355.6 mm to (0.00, -301.0)
Connections:
- removed net CC_INPUT: C30.2, IC6.6, TRIM3.2
- removed net DRUM_OUTPUT: C27.1, IC5.6, R31.1, TRIM6.3
- removed net HIGH_FREQ_WN: C36.2, IC3.6, R11.1
- removed net LOW_FREQ_WN: C35.2, IC2.6, R10.1
- removed net N$1: R15.1, R17.1, R18.2
- removed net N$10: C35.1, R15.2
- removed net N$2: IC6.2, R35.1, R36.1, R38.2
- removed net N$27: IC3.2, R11.2, R7.1
- removed net N$3: R38.1, TRIM3.1
- removed net N$32: C2.1, IC3.3, R5.1
- removed net N$33: IC2.2, R10.2, R6.1
- removed net N$34: C4.1, IC2.3, R1.2
- removed net N$36: C20.2, C22.2, D2.C, R27.2
- removed net N$37: C30.1, Q6.2, R41.1, R42.2
- removed net N$38: C32.1, Q6.3, R44.2
- removed net N$39: C31.1, C33.+, Q6.1, R43.1
- removed net N$4: IC6.5, TRIM4.1
- removed net N$40: D2.A, Q4.3, R20.2
- removed net N$41: C22.1, IC5.3, R29.2
- removed net N$42: R23.2, TRIM1.2
- removed net N$43: C25.2, IC5.2, R31.2
- removed net N$45: IC5.1, TRIM5.3
- removed net N$46: IC5.5, TRIM5.1
- removed net N$48: IC4.3, R22.1, R28.2, TRIM1.1
- removed net N$49: IC4.2, Q5.1, R21.1, R30.2
- removed net N$50: IC4.1, TRIM2.3
- removed net N$51: C19.2, D1.C, R25.2
- removed net N$52: IC4.5, TRIM2.1
- removed net N$53: D1.A, Q3.3, R19.2
- removed net N$7: IC6.1, TRIM4.3
- removed net N$8: C25.1, C27.2, R32.2
- new net BRIDGED_T_OUT: C53.1, R75.1
- new net CC_INPUT1: C54.2
- new net FILTER_OUT: C2.2
- new net N$61: IC7.3, R64.1, R65.2
- new net N$62: C49.1, R65.1
- new net N$63: C54.1, Q17.2, R76.1, R77.2
- new net N$64: D3.A, Q15.3, R66.2
- new net N$65: IC8.3, R68.2, R71.1, TRIM12.1
- new net N$66: IC8.2, Q16.1, R69.2, R70.1
- new net N$67: IC8.5, TRIM11.1
- new net N$68: IC8.1, TRIM11.3
- new net N$69: R72.2, TRIM12.2
- new net N$70: R67.1, R73.2
- new net N$71: C56.1, Q17.3, R78.2
- new net N$72: C55.1, C57.+, Q17.1, R79.1
- new net N$73: C59.2, C60.1, R81.1
- new net N$74: C60.2, Q18.2, R82.1
- new net N$75: C2.1, Q18.3, R81.2, R83.1
- net +12V: now also C52.2, IC8.7, Q15.1, Q18.1, R76.2, R79.2; no longer C11.2, C21.2, C23.1, C28.2, C9.2, IC2.7, IC3.7, IC4.7, IC5.7, IC6.7, Q3.1, Q4.1, R41.2, R43.2
- net -12V: now also C51.2, IC8.4, R77.1, R78.1, R83.2, TRIM11.2; no longer C10.2, C12.2, C24.2, C26.2, C29.2, IC2.4, IC3.4, IC4.4, IC5.4, IC6.4, R42.1, R44.1, TRIM2.2, TRIM4.2, TRIM5.2
- net AGND: now also C50.1, C51.1, C52.1, C55.2, C57.-, C58.2, Q16.3, R64.2, R66.1, R68.1, R72.1, R73.1, R80.1, R82.2; no longer C10.1, C11.1, C12.1, C19.1, C20.1, C21.1, C23.2, C24.1, C26.1, C28.1, C29.1, C31.2, C33.-, C4.2, C9.1, IC6.3, IC7.3, Q5.3, R19.1, R20.1, R23.1, R26.1, R27.1, R28.1, R29.1, R32.1, R45.1, R5.2, R6.2, R7.2, TRIM6.1
- net N$60: now also C53.2
- net OUTPUT: now also C56.2, R80.2; no longer C32.2, R45.2
- net POT1A: no longer TRIM6.2
- net POT1B: no longer R35.2
- net POT2A: no longer C36.1
- net POT2B: no longer R17.2
- net SW1: now also C58.1, C59.1, IC8.6, R69.1; no longer IC4.6, R30.1
- net SW2: no longer R36.2
- net TRIGGER: now also Q15.2; no longer Q3.2, Q4.2
- net VCA_INPUT: now also R70.2, R71.2, R74.2, R75.2; no longer R18.1, R21.2, R22.2
- net VCA_TRIGGER: now also C50.2, D3.C, Q16.2, R67.2; no longer Q5.2, R25.1, R26.2
- net WHITE_NOISE_AMP: now also R74.1; no longer C2.2, R1.1
Routing:
- net -12V: track 368.8 -> 0.00 mm, vias 7 -> 1
- net TRIGGER: track 172.3 -> 0.00 mm, vias 1 -> 0
- net SW1: track 71.4 -> 0.00 mm, vias 3 -> 0
- net CC_INPUT: track 57.9 -> 0.00 mm, vias 3 -> 0
- net OUTPUT: track 55.2 -> 0.00 mm, vias 4 -> 0
- net N$21: track 54.2 -> 0.00 mm
- net LOW_FREQ_WN: track 50.5 -> 0.00 mm
- net HIGH_FREQ_WN: track 49.7 -> 0.00 mm, vias 1 -> 0
- net WHITE_NOISE_AMP: track 48.7 -> 0.00 mm, vias 1 -> 0
- net N$32: track 37.7 -> 0.00 mm, vias 2 -> 0
- net DRUM_OUTPUT: track 34.5 -> 0.00 mm, vias 1 -> 0
- net N$43: track 32.8 -> 0.00 mm, vias 1 -> 0
- net N$37: track 32.7 -> 0.00 mm, vias 1 -> 0
- net POT2B: track 32.2 -> 0.00 mm, vias 1 -> 0
- net N$48: track 32.0 -> 0.00 mm, vias 3 -> 0
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
Commit message: Changed resistors out for shorter ones
changed resistors out for shorter ones
Parts:
- removed R54, R55: 20k, resistor:0207/10
- removed R56: 560, resistor:0207/10
- removed R57: 82k, resistor:0207/10
- removed R58, R59, R60, R61: 220k, resistor:0207/10
- removed R62, R67, R73, R80: 47k, resistor:0207/10
- removed R63, R64, R68, R69, R70, R71, R75, R76, R77, R78: 10k, resistor:0207/10
- removed R65, R83: 22k, resistor:0207/10
- removed R66: 470k, resistor:0207/10
- removed R72: 100, resistor:0207/10
- removed R74: 18k, resistor:0207/10
- removed R79: 220, resistor:0207/10
- removed R81: 2.7k, resistor:0207/10
- removed R82: 68k, resistor:0207/10
- added R1: 1k, rcl:0207/7
- added R10, R15, R18, R19, R22, R23, R31, R38, R41, R42: 10k, rcl:0207/7
- added R11, R17, R20, R21, R25: 20k, rcl:0207/7
- added R26, R30: 47k, rcl:0207/7
- added R27: 1 MEG, rcl:0207/7
- added R28, R7: 100k, rcl:0207/7
- added R29: 220k, rcl:0207/7
- added R32, R45: 22k, rcl:0207/7
- added R35: 560, rcl:0207/7
- added R36: 18k, rcl:0207/7
- added R43: 2.7k, rcl:0207/7
- added R44: 68k, rcl:0207/7
- added R5, R6: 2k, rcl:0207/7
- R12: value 4.7k -> 20k; device resistor:0207/10 -> rcl:0207/7
- R13: value 1k -> 10k; device resistor:0207/10 -> rcl:0207/7
- R14: value 100k -> 220k; device resistor:0207/10 -> rcl:0207/7
- R16: value 100k -> 20k; device resistor:0207/10 -> rcl:0207/7
- R2: value 47k -> 220k; device resistor:0207/10 -> rcl:0207/7
- R24: value 10k -> 20k; device resistor:0207/10 -> rcl:0207/7
- R3: value 2k -> 680k; device resistor:0207/10 -> rcl:0207/7
- R33, R39, R49, R52: device resistor:0207/10 -> rcl:0207/7
- R34: value 20k -> 82k; device resistor:0207/10 -> rcl:0207/7
- R37, R51: value 20k -> 10k; device resistor:0207/10 -> rcl:0207/7
- R4: value 2k -> 4.7k; device resistor:0207/10 -> rcl:0207/7
- R40: value 10k -> 100; device resistor:0207/10 -> rcl:0207/7
- R46: value 20k -> 27k; device resistor:0207/10 -> rcl:0207/7
- R47: value 20k -> 22k; device resistor:0207/10 -> rcl:0207/7
- R48: value 10k -> 470k; device resistor:0207/10 -> rcl:0207/7
- R50: value 20k -> 220; device resistor:0207/10 -> rcl:0207/7
- R53: value 10k -> 47k; device resistor:0207/10 -> rcl:0207/7
- R8: value 680k -> 10k; device resistor:0207/10 -> rcl:0207/7
- R9: value 1 MEG -> 220k; device resistor:0207/10 -> rcl:0207/7
- moved R53 976.4 mm to (1.00, -1029.0)
- moved R52 962.1 mm to (1.00, -1015.0)
- moved R51 948.0 mm to (1.00, -1001.0)
- moved R50 939.4 mm to (1.00, -987.0)
- moved R49 925.1 mm to (1.00, -973.0)
- moved R48 911.0 mm to (1.00, -959.0)
- moved R47 902.4 mm to (1.00, -945.0)
- moved R46 888.1 mm to (1.00, -931.0)
- moved R40 804.0 mm to (1.00, -847.0)
- moved R39 795.5 mm to (1.00, -833.0)
- moved R37 767.1 mm to (1.00, -805.0)
- moved R34 725.0 mm to (1.00, -763.0)
- moved R33 718.6 mm to (1.00, -749.0)
- moved R14 715.4 mm to (1.00, -679.0), turned to 0 degrees
- moved R9 701.2 mm to (1.00, -665.0), turned to 0 degrees
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Connections:
- removed net N$70: R67.1, R73.2
- new net N$1: C50.2, D3.C, R46.2
- net +12V: now also R10.2, R13.2, R15.2, R18.2, R19.2, R22.2, R23.2, R50.2, R52.2, R6.2, R8.2; no longer R24.1, R3.1, R33.1, R39.1, R40.1, R48.1, R49.1, R52.1, R53.1, R76.2, R79.2
- net -12V: now also R45.1, R49.1, R5.2, R51.1; no longer R4.2, R77.1, R78.1, R83.2
- net AGND: now also R28.2, R31.1, R33.1, R35.1, R40.1, R41.1, R44.1, R47.1, R48.1, R53.1; no longer R14.2, R56.2, R63.1, R64.2, R66.1, R68.1, R72.1, R73.1, R80.1, R82.2
- net BRIDGED_T_OUT: now also R37.1; no longer R75.1
- net N$11: now also R8.1; no longer R24.2
- net N$12: now also R11.1; no longer R34.2
- net N$13: now also R12.1; no longer R37.2
- net N$14: now also R34.1; no longer R57.1
- net N$15: now also R11.2, R12.2; no longer R34.1, R37.1
- net N$16: now also R15.1; no longer R39.2
- net N$18: now also R16.1; no longer R46.2
- net N$19: now also R17.1; no longer R47.2
- net N$20: now also R3.1; no longer R8.2
- net N$21: now also R1.1, R5.1, R7.1; no longer R13.2, R16.2, R4.1
- net N$22: now also R14.2, R2.2, R29.2, R30.1, R9.2; no longer R58.2, R59.2, R60.2, R61.2, R62.1
- net N$23: now also R26.1, R27.2; no longer R2.1, R9.2
- net N$28: now also R26.2; no longer R2.2
- net N$29: now also R16.2, R17.2; no longer R46.1, R47.1
- net N$30: now also R4.1; no longer R12.2
- net N$31: now also R18.1; no longer R48.2
- net N$35: now also R20.1; no longer R50.2
- net N$44: now also R21.1; no longer R51.2
- net N$47: now also R35.2; no longer R56.1
- net N$5: now also R1.2; no longer R13.1
- net N$54: now also R20.2, R21.2; no longer R50.1, R51.1
- net N$55: now also R22.1; no longer R52.2
- net N$56: now also R24.1; no longer R54.2
- net N$57: now also R25.1; no longer R55.2
- net N$58: now also R30.2, R31.2; no longer R62.2, R63.2
- net N$59: now also R24.2, R25.2; no longer R54.1, R55.1
- net N$6: now also R4.2, R6.1; no longer R12.1, R8.1
- net N$60: now also R34.2; no longer R57.2
- net N$61: now also R32.2, R33.2; no longer R64.1, R65.2
- net N$62: now also R32.1; no longer R65.1
- net N$63: now also R51.2, R52.1; no longer R76.1, R77.2
- net N$64: now also R48.2; no longer R66.2
- net N$65: now also R39.2, R41.2; no longer R68.2, R71.1
- net N$66: now also R38.2, R42.1; no longer R69.2, R70.1
- net N$69: now also R40.2; no longer R72.2
- net N$71: now also R49.2; no longer R78.2
- net N$72: now also R50.1; no longer R79.1
- net N$73: now also R43.2; no longer R81.1
- net N$74: now also R44.2; no longer R82.1
- net N$75: now also R43.1, R45.2; no longer R81.2, R83.1
- net N$9: now also R27.1; no longer R9.1
- net OSC1: now also R10.1, R2.1; no longer R33.2, R58.1
- net OSC2: now also R13.1, R9.1; no longer R40.2, R59.1
- net OSC3: now also R14.1, R19.1; no longer R49.2, R60.1
- net OSC4: now also R23.1, R29.1; no longer R53.2, R61.1
- net OUTPUT: now also R53.2; no longer R80.2
- net SW1: now also R42.2; no longer R69.1
- net VCA_INPUT: now also R36.2, R37.2, R38.1, R39.1; no longer R70.2, R71.2, R74.2, R75.2
- net VCA_TRIGGER: now also R46.1, R47.2; no longer C50.2, D3.C, R67.2
- net WHITE_NOISE: now also R7.2; no longer R16.1
- net WHITE_NOISE_AMP: now also R28.1, R36.1; no longer R14.1, R74.1
