File: Hi Hat/PCB/Hi-Hat2.sch (EAGLE design)
At the start: 132 parts, among them IC1 LM741P, IC2 LM741P, IC3 LM741P, IC7 LM741P, IC8 LM741P, Q1 2N3904, Q10 2N2222A, Q11 2N2222A, Q12 2N2222A, Q13 2N2222A, Q14 2N2222A, Q15 2N2222A, Q17 2N3904, Q18 2N3904, Q2 2N3904, Q7 2N2222A, Q8 2N2222A, Q9 2N2222A

Commit message: Updates to cymbals
Parts:
- removed TRIM12: 20 OHM, rcl:R-TRIMM64W
- added C19, C20, C21, C22, C23: 0.1uF, resistor:C-EU050-024X044
- added D1, D2, D4, D5: 200mA/100V/1V, SparkFun-DiscreteSemi:DIODE-1N4148
- added IC4, IC5: LM741P, linear:LM741P
- added Q5: (no value), Capstone:J176
- added R60: 470k, rcl:R-US_0207/7
- added R61: 100k, rcl:R-US_0207/7
- R36: value 18k -> 300k
- R40: value 100 -> 10k
- R56: value 10k -> 220k
Connections:
- removed net N$69: R40.2, TRIM12.S
- removed net VCA_INPUT: R36.2, R37.2, R38.1, R39.1
- new net CYMBAL_SIGNAL: D1.C, D2.A, R60.1
- new net N$32: IC4.-IN, R36.1, R37.2
- new net N$34: C21.1, R37.1
- new net N$36: C21.2, IC8.OUT, R42.2
- new net N$37: IC5.OUT, R40.2
- new net N$38: D4.C, D5.A, IC4.OUT, R36.2
- new net N$39: D1.A, D2.C, IC3.OUT, R56.2
- new net WN_SIGNAL: D4.A, D5.C, R61.1
- net +12V: now also C20.2, C23.2, IC4.V+, IC5.V+
- net -12V: now also C19.2, C22.2, IC4.V-, IC5.V-
- net AGND: now also C19.1, C20.1, C22.1, C23.1, IC4.+IN, IC5.+IN, Q5.G, Q5.S; no longer R40.1
- net BRIDGED_T_OUT: no longer R37.1
- net N$10: now also IC5.-IN, R40.1, R60.2, R61.2; no longer IC3.OUT, R56.2
- net N$65: now also Q5.D; no longer TRIM12.A
- net SW1: no longer IC8.OUT, R42.2
- net WHITE_NOISE_AMP: now also R38.1, R39.1; no longer R36.1
Other:
- moved on the sheet: C2, C58, C59, C60, Q18, R36, R37, R40, R43, R44, R45
