File: Hi Hat/PCB/Waveform Generator Board.brd (EAGLE design)
At the start: 100 x 50 mm, 145 parts, among them IC1 LM741P, IC2 LM741P, IC3 LM741P, IC4 LM741P, IC5 LM741P, IC7 LM741P, IC8 LM741P, Q1 2N3904, Q10 2N2222A, Q11 2N2222A, Q12 2N2222A, Q13 2N2222A, Q14 2N2222A, Q15 2N2222A, Q17 2N3904, Q18 2N3904, Q2 2N3904, Q7 2N2222A, Q8 2N2222A, Q9 2N2222A

Commit message: Created Waveform generator board
Parts:
- removed C34, C37, C38, C39, C40, C45, C46, C51, C52: 0.1uF, resistor:C050-024X044
- removed C41, C42: 47nF, resistor:C050-024X044
- removed C43, C44: 33nF, resistor:C050-024X044
- removed C47, C48: 3.3nF, resistor:C050-024X044
- removed C49, C59, C60: 1nF, resistor:C050-024X044
- removed C50: 0.47uF, resistor:C050-024X044
- removed C53: 22nF, resistor:C050-024X044
- removed C54, C56: 2.2u, resistor:C050-024X044
- removed C55: 1u, resistor:C050-024X044
- removed C57: 10uF, rcl:E2,5-6
- removed C58: 1.5nF, resistor:C050-024X044
- removed D1, D2, D3, D4, D5: 200mA/100V/1V, SparkFun-DiscreteSemi:DIODE-1N4148
- removed IC2, IC3, IC4, IC5, IC7, IC8: LM741P, linear:DIL08
- removed Q13, Q14, Q15: 2N2222A, SparkFun-DiscreteSemi:TO-92
- removed Q16: (no value), Capstone:TO-92
- removed Q17, Q18: 2N3904, transistor:TO92
- removed R16, R21: 20k, rcl:0207/7
- removed R26: 68k, rcl:0207/7
- removed R31, R49, R51, R52, R54, R55, R57, R58, R59: 10k, rcl:0207/7
- removed R45, R47: 22k, rcl:0207/7
- removed R46: 27k, rcl:0207/7
- removed R48, R60: 470k, rcl:0207/7
- removed R50: 220, rcl:0207/7
- removed R53: 47k, rcl:0207/7
- removed R56: 220k, rcl:0207/7
- removed R61: 100k, rcl:0207/7
- removed TRIM10, TRIM11, TRIM7, TRIM8, TRIM9: 10k, rcl:RTRIM64W
- added C24: 33nF, resistor:C050-024X044
- added C25, C27: 2.2u, resistor:C050-024X044
- added C26: 1u, resistor:C050-024X044
- added C28: 10uF, rcl:E2,5-6
- added J1: (no value), SparkFun-Connectors:2X3-NS
- added J2, J3, J4, J5, J6: (no value), SparkFun-Connectors:1X03_NO_SILK
- added J7, J8: (no value), SparkFun-Connectors:1X02_NO_SILK
- added Q6: 2N2222A, SparkFun-DiscreteSemi:TO-92
- added TRIM2, TRIM3, TRIM4: 10k, rcl:RTRIM64W
- C1, C2, C5, C8, C9: value 0.1uF -> 10uF; device resistor:C050-024X044 -> rcl:E2,5-6
- C13, C15: value 10uF -> 2.2u; device rcl:E2,5-6 -> resistor:C050-024X044
- C14, C3: value 10uF -> 1u; device rcl:E2,5-6 -> resistor:C050-024X044
- C17, C18: value 1u -> 0.1uF
- C21, C22: value 0.1uF -> 47nF
- C23: value 0.1uF -> 33nF
- C4: value 0.1uF -> 1u
- Q1, Q2: value 2N3904 -> 2N2222A; device transistor:TO92 -> SparkFun-DiscreteSemi:TO-92
- Q10, Q11, Q12, Q9: value 2N2222A -> 2N3904; device SparkFun-DiscreteSemi:TO-92 -> transistor:TO92
- Q3, Q4, Q5: value (none) -> 2N2222A; device Capstone:TO-92 -> SparkFun-DiscreteSemi:TO-92
- R1: value 1k -> 2k
- R11: value 20k -> 220
- R12, R24: value 20k -> 10k
- R13, R38: value 10k -> 47k
- R14, R29, R9: value 220k -> 10k
- R15, R22: value 10k -> 20k
- R2: value 220k -> 2k
- R27: value 100k -> 20k
- R28: value 100k -> 10k
- R30: value 47k -> 20k
- R32: value 22k -> 20k
- R34: value 82k -> 220k
- R35: value 560 -> 220k
- R36: value 300k -> 220k
- R37: value 10k -> 220k
- R42: value 10k -> 220
- R43: value 2.7k -> 10k
- R44: value 68k -> 47k
- R5: value 2k -> 1k
- R6: value 2k -> 100k
- R7: value 100k -> 68k
- R8: value 10k -> 100k
- moved C21 1158.2 mm to (70.0, 29.0)
- moved Q5 1135.6 mm to (78.0, 23.0), turned to 270 degrees
- moved C12 1135.1 mm to (11.0, 43.0), turned to 270 degrees
- moved Q4 1071.3 mm to (53.0, 23.0), turned to 270 degrees
- moved R44 925.4 mm to (91.0, 18.0)
- moved R43 907.5 mm to (91.0, 14.0)
- moved R42 884.6 mm to (81.0, 6.00)
- moved R41 874.7 mm to (81.0, 10.0)
- moved R39 854.8 mm to (81.0, 18.0), turned to 180 degrees
- moved R38 824.0 mm to (71.0, 2.00), turned to 180 degrees
- moved R35 794.1 mm to (71.0, 14.0)
- moved R33 792.0 mm to (98.0, 37.0), turned to 90 degrees
- moved R34 784.1 mm to (71.0, 18.0)
- moved R32 777.1 mm to (90.0, 37.0), turned to 90 degrees
- moved R30 748.8 mm to (86.0, 37.0), turned to 90 degrees
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Connections:
- removed net BRIDGED_T_OUT: C53.1
- removed net CC_INPUT1: C54.2
- removed net CYMBAL_SIGNAL: D1.C, D2.A, R60.1
- removed net FILTER_OUT: C2.2
- removed net N$1: C50.2, D3.C, R46.2
- removed net N$10: IC5.2, R40.1, R60.2, R61.2
- removed net N$14: C47.2, IC7.2, R34.1
- removed net N$27: C12.1, R59.1
- removed net N$32: IC4.2, R36.1, R37.2
- removed net N$34: C21.1, R37.1
- removed net N$36: C21.2, IC8.6, R42.2
- removed net N$37: IC5.6, R40.2
- removed net N$38: D4.C, D5.A, IC4.6, R36.2
- removed net N$39: D1.A, D2.C, IC3.6, R56.2
- removed net N$47: C47.1, C48.2, R35.2
- removed net N$60: C48.1, C53.2, IC7.6, R34.2
- removed net N$61: IC7.3, R32.2, R33.2
- removed net N$62: C49.1, R32.1
- removed net N$64: D3.A, Q15.3, R48.2
- removed net N$65: IC8.3, Q5.1, R39.2, R41.2
- removed net N$66: IC8.2, Q16.1, R38.2, R42.1
- removed net N$67: IC8.5, TRIM11.1
- removed net N$68: IC8.1, TRIM11.3
- removed net N$7: IC2.1, TRIM1.3
- removed net N$73: C59.2, C60.1, R43.2
- removed net N$74: C60.2, Q18.2, R44.2
- removed net N$75: C2.1, Q18.3, R43.1, R45.2
- removed net N$8: IC3.2, R56.1, R59.2
- removed net SW4: C12.2, IC2.6, R58.2
- removed net VCA_INPUT1: R54.1, R55.1
- removed net VCA_TRIGGER: Q16.2, Q3.2, R46.1, R47.2
- removed net WHITE_NOISE_AMP: C34.1, R28.1, R38.1, R39.1
- removed net WN_SIGNAL: D4.A, D5.C, R61.1
- new net SQUARE_WAVE_BUFFERED: C27.2, J1.2, R44.2
- new net WHITE_NOISE_BUFFERED: C15.2, J1.4, R13.2
- net +12V: now also C1.+, C3.2, R1.2, R11.2, R14.2, R24.2, R28.2, R29.2, R33.2, R40.2, R42.2, R9.2, TRIM1.3, TRIM2.3, TRIM3.3, TRIM4.3; no longer C15.+, C17.2, C20.2, C23.2, C46.2, C52.2, C7.2, C9.2, IC2.7, IC3.7, IC4.7, IC5.7, IC7.7, IC8.7, Q15.1, Q18.1, R10.2, R13.2, R15.2, R22.2, R50.2, R52.2, R6.2, R8.2, TRIM10.3, TRIM7.3, TRIM8.3, TRIM9.3
- net -12V: now also C12.2, C2.-, C4.1, R10.1, R12.1, R2.2, R41.1, R43.1; no longer C10.2, C16.-, C18.1, C19.2, C22.2, C4.2, C45.2, C51.2, C8.2, IC2.4, IC3.4, IC4.4, IC5.4, IC7.4, IC8.4, R45.1, R49.1, R5.2, R51.1, TRIM1.2, TRIM11.2
- net AGND: now also C1.-, C12.1, C14.2, C16.-, C2.+, C26.2, C28.-, C3.1, C4.2, Q1.3, Q2.3, Q6.3, R13.1, R39.1; no longer C10.1, C15.-, C16.+, C17.1, C18.2, C19.1, C20.1, C22.1, C23.1, C4.1, C45.1, C46.1, C50.1, C51.1, C52.1, C55.2, C57.-, C58.2, C7.1, C8.1, C9.1, IC3.3, IC4.3, IC5.3, Q10.3, Q11.3, Q12.3, Q13.3, Q14.3, Q16.3, Q4.2, Q5.2, Q9.3, R28.2, R31.1, R33.1, R35.1, R41.1, R47.1, R48.1, R53.1, R57.1
- net N$11: now also C17.2, Q1.1, R14.1; no longer C37.2, Q8.1, R8.1
- net N$12: now also C17.1, Q2.2, R15.1; no longer C37.1, Q7.2, R11.1
- net N$13: now also C18.2, Q1.2, R17.1; no longer C38.2, Q8.2, R12.1
- net N$15: now also R15.2, R17.2, TRIM1.2; no longer R11.2, R12.2, TRIM7.2
- net N$16: now also C19.2, Q3.1, R19.1; no longer C39.2, Q10.1, R15.1
- net N$17: now also Q10.2, Q11.2; no longer Q1.2, Q2.2
- net N$18: now also C19.1, Q4.2, R20.1; no longer C39.1, Q9.2, R16.1
- net N$19: now also C20.2, Q3.2, R22.1; no longer C40.2, Q10.2, R17.1
- net N$2: now also C13.1, Q12.2, R10.2, R9.1; no longer IC2.3, Q4.1, R55.2, R57.2
- net N$20: now also C7.1, Q10.3; no longer C6.1, Q1.3
- net N$21: now also C5.-, C6.1, C9.-, R2.1, R6.1; no longer C14.-, C3.-, C5.1, R1.1, R7.1
- net N$22: now also R34.2, R35.2, R36.2, R37.2, R38.1; no longer R14.2, R2.2, R29.2, R30.1, R9.2
- net N$23: now also R7.1, R8.2; no longer R26.1, R27.2
- net N$28: now also C10.1, R7.2; no longer C1.1, R26.2
- net N$29: now also R20.2, R22.2, TRIM2.2; no longer R16.2, R17.2, TRIM8.2
- net N$3: now also C15.1, Q12.3, R12.2; no longer IC2.2, Q3.1, R54.2, R58.1
- net N$30: now also C8.+, Q11.1; no longer C13.+, Q2.1
- net N$31: now also C21.2, Q5.1, R24.1; no longer C41.2, Q12.1, R18.1
- net N$35: now also C21.1, Q6.2, R25.1; no longer C41.1, Q11.2, R20.1
- net N$4: now also C14.1, C16.+, Q12.1, R11.1; no longer IC2.5, TRIM1.1
- net N$44: now also C22.2, Q5.2, R27.1; no longer C42.2, Q12.2, R21.1
- net N$5: now also C9.+, Q11.3, R5.2; no longer C14.+, Q2.3, R1.2
- net N$54: now also R25.2, R27.2, TRIM3.2; no longer R20.2, R21.2, TRIM9.2
- net N$55: now also C23.2, Q7.1, R29.1; no longer C43.2, Q14.1, R22.1
- net N$56: now also C23.1, Q8.2, R30.1; no longer C43.1, Q13.2, R24.1
- net N$57: now also C24.2, Q7.2, R32.1; no longer C44.2, Q14.2, R25.1
- net N$58: now also C25.2, R38.2, R39.2; no longer C49.2, R30.2, R31.2
- net N$59: now also R30.2, R32.2, TRIM4.2; no longer R24.2, R25.2, TRIM10.2
- net N$6: now also C5.+, C7.2, R1.1; no longer C3.+, C5.2, R6.1
- net N$63: now also C25.1, Q9.2, R40.1, R41.2; no longer C54.1, Q17.2, R51.2, R52.1
- net N$71: now also C27.1, Q9.3, R43.2; no longer C56.1, Q17.3, R49.2
- net N$72: now also C26.1, C28.+, Q9.1, R42.1; no longer C55.1, C57.+, Q17.1, R50.1
- net N$9: now also C13.2, R8.1; no longer C34.2, R27.1
- net OSC1: now also C18.1, Q2.1, R18.1, R34.1; no longer C38.1, Q7.1, R10.1, R2.1
- net OSC2: now also C20.1, Q4.1, R23.1, R35.1; no longer C40.1, Q9.1, R13.1, R9.1
- net OSC3: now also C22.1, Q6.1, R28.1, R36.1; no longer C42.1, Q11.1, R14.1, R19.1
- net OSC4: now also C24.1, Q8.1, R33.1, R37.1; no longer C44.1, Q13.1, R23.1, R29.1
- net OUTPUT: no longer C56.2, R53.2
- net SW1: no longer C58.1, C59.1
- net TRIGGER: no longer Q15.2
- net WHITE_NOISE: now also C10.2, C8.-, R6.2; no longer C1.2, C13.-, R7.2
Routing:
- net OSC4: track 0.00 -> 48.7 mm
- net OSC1: track 0.00 -> 47.1 mm
- net N$6: track 0.73 -> 46.7 mm, vias 0 -> 1
- net OSC2: track 0.00 -> 37.2 mm
- net WHITE_NOISE: track 0.00 -> 36.0 mm
- net N$21: track 0.00 -> 35.4 mm
- net OSC3: track 0.00 -> 32.8 mm
- net N$4: track 0.00 -> 27.7 mm
- net N$58: track 0.00 -> 26.6 mm
- net N$63: track 0.00 -> 25.5 mm, vias 0 -> 1
- net N$72: track 0.00 -> 25.4 mm
- net -12V: track 0.00 -> 25.2 mm, vias 1 -> 0
- net N$2: track 0.00 -> 24.7 mm
- net N$3: track 0.00 -> 23.1 mm
- net N$28: track 0.00 -> 21.1 mm
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Other:
- board text added: "Cymbal Waveform PCB March 16, 2019"
- board text added: "SQ"
- board text added: "WN"
- board text removed: "Snare Drum March 4, 2019"
