File: Hi Hat/PCB/Waveform Generator Board.sch (EAGLE design)
At the start: 132 parts, among them IC1 LM741P, IC2 LM741P, IC3 LM741P, IC7 LM741P, IC8 LM741P, Q1 2N3904, Q10 2N2222A, Q11 2N2222A, Q12 2N2222A, Q13 2N2222A, Q14 2N2222A, Q15 2N2222A, Q17 2N3904, Q18 2N3904, Q2 2N3904, Q7 2N2222A, Q8 2N2222A, Q9 2N2222A

Commit message: Created Waveform generator board
Parts:
- removed C34, C37, C38, C39, C40, C45, C46, C51, C52: 0.1uF, resistor:C-EU050-024X044
- removed C41, C42: 47nF, resistor:C-EU050-024X044
- removed C43, C44: 33nF, resistor:C-EU050-024X044
- removed C47, C48: 3.3nF, resistor:C-EU050-024X044
- removed C49, C59, C60: 1nF, resistor:C-EU050-024X044
- removed C50: 0.47uF, resistor:C-EU050-024X044
- removed C53: 22nF, resistor:C-EU050-024X044
- removed C54, C56: 2.2u, resistor:C-EU050-024X044
- removed C55: 1u, resistor:C-EU050-024X044
- removed C57: 10uF, rcl:CPOL-USE2.5-6
- removed C58: 1.5nF, resistor:C-EU050-024X044
- removed D3: 200mA/100V/1V, SparkFun-DiscreteSemi:DIODE-1N4148
- removed IC2, IC3, IC7, IC8: LM741P, linear:LM741P
- removed Q13, Q14, Q15: 2N2222A, SparkFun-DiscreteSemi:TRANS_NPN-P2N2222A
- removed Q16: (no value), Capstone:J176
- removed Q17, Q18: 2N3904, transistor:2N3904
- removed R16, R21: 20k, rcl:R-US_0207/7
- removed R26: 68k, rcl:R-US_0207/7
- removed R31, R49, R51, R52, R54, R55, R56, R57, R58, R59: 10k, rcl:R-US_0207/7
- removed R45, R47: 22k, rcl:R-US_0207/7
- removed R46: 27k, rcl:R-US_0207/7
- removed R48: 470k, rcl:R-US_0207/7
- removed R50: 220, rcl:R-US_0207/7
- removed R53: 47k, rcl:R-US_0207/7
- removed TRIM10, TRIM11, TRIM7, TRIM8, TRIM9: 10k, rcl:R-TRIMM64W
- removed TRIM12: 20 OHM, rcl:R-TRIMM64W
- added C19, C20: 0.1uF, resistor:C-EU050-024X044
- added C21, C22: 47nF, resistor:C-EU050-024X044
- added C23, C24: 33nF, resistor:C-EU050-024X044
- added C25, C27: 2.2u, resistor:C-EU050-024X044
- added C26: 1u, resistor:C-EU050-024X044
- added C28: 10uF, rcl:CPOL-USE2.5-6
- added J1: (no value), SparkFun-Connectors:CONN_03X2NO_SILK
- added J2, J3, J4, J5, J6: (no value), SparkFun-Connectors:CONN_031X03_NO_SILK
- added J7, J8: (no value), SparkFun-Connectors:CONN_021X02_NO_SILK
- added Q5, Q6: 2N2222A, SparkFun-DiscreteSemi:TRANS_NPN-P2N2222A
- added TRIM2, TRIM3, TRIM4: 10k, rcl:R-TRIMM64W
- C1, C2, C5, C8, C9: value 0.1uF -> 10uF; device resistor:C-EU050-024X044 -> rcl:CPOL-USE2.5-6
- C13, C15: value 10uF -> 2.2u; device rcl:CPOL-USE2.5-6 -> resistor:C-EU050-024X044
- C14, C3: value 10uF -> 1u; device rcl:CPOL-USE2.5-6 -> resistor:C-EU050-024X044
- C17, C18: value 1u -> 0.1uF
- C4: value 0.1uF -> 1u
- Q1, Q2: value 2N3904 -> 2N2222A; device transistor:2N3904 -> SparkFun-DiscreteSemi:TRANS_NPN-P2N2222A
- Q10, Q11, Q12, Q9: value 2N2222A -> 2N3904; device SparkFun-DiscreteSemi:TRANS_NPN-P2N2222A -> transistor:2N3904
- Q3, Q4: value (none) -> 2N2222A; device Capstone:J176 -> SparkFun-DiscreteSemi:TRANS_NPN-P2N2222A
- R1: value 1k -> 2k
- R11: value 20k -> 220
- R12, R24: value 20k -> 10k
- R13, R38: value 10k -> 47k
- R14, R29, R9: value 220k -> 10k
- R15, R22: value 10k -> 20k
- R2: value 220k -> 2k
- R27: value 100k -> 20k
- R28: value 100k -> 10k
- R30: value 47k -> 20k
- R32: value 22k -> 20k
- R34: value 82k -> 220k
- R35: value 560 -> 220k
- R36: value 18k -> 220k
- R37: value 10k -> 220k
- R40: value 100 -> 10k
- R42: value 10k -> 220
- R43: value 2.7k -> 10k
- R44: value 68k -> 47k
- R5: value 2k -> 1k
- R6: value 2k -> 100k
- R7: value 100k -> 68k
- R8: value 10k -> 100k
Connections:
- removed net BRIDGED_T_OUT: C53.1, R37.1
- removed net CC_INPUT1: C54.2
- removed net FILTER_OUT: C2.2
- removed net N$1: C50.2, D3.C, R46.2
- removed net N$10: IC3.OUT, R56.2
- removed net N$14: C47.2, IC7.-IN, R34.1
- removed net N$27: C12.1, R59.1
- removed net N$47: C47.1, C48.2, R35.2
- removed net N$60: C48.1, C53.2, IC7.OUT, R34.2
- removed net N$61: IC7.+IN, R32.2, R33.2
- removed net N$62: C49.1, R32.1
- removed net N$64: D3.A, Q15.E, R48.2
- removed net N$65: IC8.+IN, R39.2, R41.2, TRIM12.A
- removed net N$66: IC8.-IN, Q16.D, R38.2, R42.1
- removed net N$67: IC8.ON2, TRIM11.A
- removed net N$68: IC8.ON1, TRIM11.E
- removed net N$69: R40.2, TRIM12.S
- removed net N$7: IC2.ON1, TRIM1.E
- removed net N$73: C59.2, C60.1, R43.2
- removed net N$74: C60.2, Q18.B, R44.2
- removed net N$75: C2.1, Q18.E, R43.1, R45.2
- removed net N$8: IC3.-IN, R56.1, R59.2
- removed net SW4: C12.2, IC2.OUT, R58.2
- removed net VCA_INPUT: R36.2, R37.2, R38.1, R39.1
- removed net VCA_INPUT1: R54.1, R55.1
- removed net VCA_TRIGGER: Q16.G, Q3.G, R46.1, R47.2
- removed net WHITE_NOISE_AMP: C34.1, R28.1, R36.1
- new net SQUARE_WAVE_BUFFERED: C27.2, J1.2, R44.2
- new net WHITE_NOISE_BUFFERED: C15.2, J1.4, R13.2
- net +12V: now also C1.+, C3.2, R1.2, R11.2, R14.2, R24.2, R28.2, R29.2, R33.2, R40.2, R42.2, R9.2, TRIM1.E, TRIM2.E, TRIM3.E, TRIM4.E; no longer C15.+, C17.2, C46.2, C52.2, C7.2, C9.2, IC2.V+, IC3.V+, IC7.V+, IC8.V+, Q15.C, Q18.C, R10.2, R13.2, R15.2, R22.2, R50.2, R52.2, R6.2, R8.2, TRIM10.E, TRIM7.E, TRIM8.E, TRIM9.E
- net -12V: now also C12.2, C2.-, C4.1, R10.1, R12.1, R2.2, R41.1, R43.1; no longer C10.2, C16.-, C18.1, C4.2, C45.2, C51.2, C8.2, IC2.V-, IC3.V-, IC7.V-, IC8.V-, R45.1, R49.1, R5.2, R51.1, TRIM1.S, TRIM11.S
- net AGND: now also C1.-, C12.1, C14.2, C16.-, C2.+, C26.2, C28.-, C3.1, C4.2, Q1.E, Q2.E, Q3.E, Q4.E, Q5.E, Q6.E, R13.1, R39.1; no longer C10.1, C15.-, C16.+, C17.1, C18.2, C4.1, C45.1, C46.1, C50.1, C51.1, C52.1, C55.2, C57.-, C58.2, C7.1, C8.1, C9.1, IC3.+IN, Q10.E, Q11.E, Q12.E, Q13.E, Q14.E, Q16.S, Q3.S, Q4.G, Q4.S, Q9.E, R28.2, R31.1, R33.1, R35.1, R40.1, R41.1, R47.1, R48.1, R53.1, R57.1
- net N$11: now also C17.2, Q1.C, R14.1; no longer C37.2, Q8.C, R8.1
- net N$12: now also C17.1, Q2.B, R15.1; no longer C37.1, Q7.B, R11.1
- net N$13: now also C18.2, Q1.B, R17.1; no longer C38.2, Q8.B, R12.1
- net N$15: now also R15.2, R17.2, TRIM1.S; no longer R11.2, R12.2, TRIM7.S
- net N$16: now also C19.2, Q3.C, R19.1; no longer C39.2, Q10.C, R15.1
- net N$17: now also Q10.B, Q11.B; no longer Q1.B, Q2.B
- net N$18: now also C19.1, Q4.B, R20.1; no longer C39.1, Q9.B, R16.1
- net N$19: now also C20.2, Q3.B, R22.1; no longer C40.2, Q10.B, R17.1
- net N$2: now also C13.1, Q12.B, R10.2, R9.1; no longer IC2.+IN, Q4.D, R55.2, R57.2
- net N$20: now also C7.1, Q10.E; no longer C6.1, Q1.E
- net N$21: now also C5.-, C6.1, C9.-, R2.1, R6.1; no longer C14.-, C3.-, C5.1, R1.1, R7.1
- net N$22: now also R34.2, R35.2, R36.2, R37.2, R38.1; no longer R14.2, R2.2, R29.2, R30.1, R9.2
- net N$23: now also R7.1, R8.2; no longer R26.1, R27.2
- net N$28: now also C10.1, R7.2; no longer C1.1, R26.2
- net N$29: now also R20.2, R22.2, TRIM2.S; no longer R16.2, R17.2, TRIM8.S
- net N$3: now also C15.1, Q12.E, R12.2; no longer IC2.-IN, Q3.D, R54.2, R58.1
- net N$30: now also C8.+, Q11.C; no longer C13.+, Q2.C
- net N$31: now also C21.2, Q5.C, R24.1; no longer C41.2, Q12.C, R18.1
- net N$35: now also C21.1, Q6.B, R25.1; no longer C41.1, Q11.B, R20.1
- net N$4: now also C14.1, C16.+, Q12.C, R11.1; no longer IC2.ON2, TRIM1.A
- net N$44: now also C22.2, Q5.B, R27.1; no longer C42.2, Q12.B, R21.1
- net N$5: now also C9.+, Q11.E, R5.2; no longer C14.+, Q2.E, R1.2
- net N$54: now also R25.2, R27.2, TRIM3.S; no longer R20.2, R21.2, TRIM9.S
- net N$55: now also C23.2, Q7.C, R29.1; no longer C43.2, Q14.C, R22.1
- net N$56: now also C23.1, Q8.B, R30.1; no longer C43.1, Q13.B, R24.1
- net N$57: now also C24.2, Q7.B, R32.1; no longer C44.2, Q14.B, R25.1
- net N$58: now also C25.2, R38.2, R39.2; no longer C49.2, R30.2, R31.2
- net N$59: now also R30.2, R32.2, TRIM4.S; no longer R24.2, R25.2, TRIM10.S
- net N$6: now also C5.+, C7.2, R1.1; no longer C3.+, C5.2, R6.1
- net N$63: now also C25.1, Q9.B, R40.1, R41.2; no longer C54.1, Q17.B, R51.2, R52.1
- net N$71: now also C27.1, Q9.E, R43.2; no longer C56.1, Q17.E, R49.2
- net N$72: now also C26.1, C28.+, Q9.C, R42.1; no longer C55.1, C57.+, Q17.C, R50.1
- net N$9: now also C13.2, R8.1; no longer C34.2, R27.1
- net OSC1: now also C18.1, Q2.C, R18.1, R34.1; no longer C38.1, Q7.C, R10.1, R2.1
- net OSC2: now also C20.1, Q4.C, R23.1, R35.1; no longer C40.1, Q9.C, R13.1, R9.1
- net OSC3: now also C22.1, Q6.C, R28.1, R36.1; no longer C42.1, Q11.C, R14.1, R19.1
- net OSC4: now also C24.1, Q8.C, R33.1, R37.1; no longer C44.1, Q13.C, R23.1, R29.1
- net OUTPUT: no longer C56.2, R53.2
- net SW1: no longer C58.1, C59.1, IC8.OUT, R42.2
- net TRIGGER: no longer Q15.B
- net WHITE_NOISE: now also C10.2, C8.-, R6.2; no longer C1.2, C13.-, R7.2
Other:
- note added: "White Noise Amplifier / Buffer"
- note removed: "White Noise Amplifier"
- moved on the sheet: C10, C11, C12, C16, C17, C18, C4, C6, C7, IC1, Q7, Q8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
