File: Hi Hat/PCB/Hi-Hat.sch (EAGLE design)
At the start: 150 parts, among them IC1 LM741P, IC2 LM741P, IC3 LM741P, IC4 LM741P, IC5 LM741P, IC6 LM741P, IC7 LM741P, Q1 2N3904, Q10 2N2222A, Q11 2N2222A, Q12 2N2222A, Q13 2N2222A, Q14 2N2222A, Q2 2N3904, Q3 2N2222A, Q4 2N2222A, Q6 2N3904, Q7 2N2222A, Q8 2N2222A, Q9 2N2222A

Commit message: Completed most of hi-hat schematic
Parts:
- removed C10, C11, C12, C21, C22, C23, C24, C26, C28, C29, C35, C36, C9: 0.1uF, resistor:C-EU050-024X044
- removed C19, C20: 0.33uF, resistor:C-EU050-024X044
- removed C25, C27: 33nF, resistor:C-EU050-024X044
- removed C30, C32: 2.2u, resistor:C-EU050-024X044
- removed C31: 1u, resistor:C-EU050-024X044
- removed C33: 10uF, rcl:CPOL-USE2.5-6
- removed C4: 1nF, resistor:C-EU050-024X044
- removed D1, D2: 200mA/100V/1V, SparkFun-DiscreteSemi:DIODE-1N4148
- removed IC2, IC3, IC4, IC5, IC6: LM741P, linear:LM741P
- removed J1, J2: (no value), SparkFun-Connectors:CONN_03X2NO_SILK
- removed J3, J4: (no value), SparkFun-Connectors:CONN_021X02_NO_SILK
- removed Q3, Q4: 2N2222A, SparkFun-DiscreteSemi:TRANS_NPN-P2N2222A
- removed Q5: (no value), Capstone:J176
- removed Q6: 2N3904, transistor:2N3904
- removed R1, R5: 15k, resistor:R-US_0207/10
- removed R10, R15, R17, R18, R21, R22, R28, R30, R35, R36, R41, R42, R44: 10k, resistor:R-US_0207/10
- removed R11, R6: 2k, resistor:R-US_0207/10
- removed R19, R20: 470k, resistor:R-US_0207/10
- removed R23: 100, resistor:R-US_0207/10
- removed R25: 51k, resistor:R-US_0207/10
- removed R26, R45: 47k, resistor:R-US_0207/10
- removed R27: 100k, resistor:R-US_0207/10
- removed R29, R32, R38: 1k, resistor:R-US_0207/10
- removed R31: 1meg, resistor:R-US_0207/10
- removed R43: 220, resistor:R-US_0207/10
- removed R7: 4.7k, resistor:R-US_0207/10
- removed TRIM1: 20 OHM, rcl:R-TRIMM64W
- removed TRIM2, TRIM3, TRIM4, TRIM5, TRIM6: 10k, rcl:R-TRIMM64W
- added C50: 0.47uF, resistor:C-EU050-024X044
- added C51, C52: 0.1uF, resistor:C-EU050-024X044
- added C53: 22nF, resistor:C-EU050-024X044
- added C54, C56: 2.2u, resistor:C-EU050-024X044
- added C55: 1u, resistor:C-EU050-024X044
- added C57: 10uF, rcl:CPOL-USE2.5-6
- added C58: 1.5nF, resistor:C-EU050-024X044
- added C59, C60: 1nF, resistor:C-EU050-024X044
- added D3: 200mA/100V/1V, SparkFun-DiscreteSemi:DIODE-1N4148
- added IC8: LM741P, linear:LM741P
- added Q15: 2N2222A, SparkFun-DiscreteSemi:TRANS_NPN-P2N2222A
- added Q16: (no value), Capstone:J176
- added Q17, Q18: 2N3904, transistor:2N3904
- added R64, R68, R69, R70, R71, R75, R76, R77, R78: 10k, resistor:R-US_0207/10
- added R65, R83: 22k, resistor:R-US_0207/10
- added R66: 470k, resistor:R-US_0207/10
- added R67, R73, R80: 47k, resistor:R-US_0207/10
- added R72: 100, resistor:R-US_0207/10
- added R74: 18k, resistor:R-US_0207/10
- added R79: 220, resistor:R-US_0207/10
- added R81: 2.7k, resistor:R-US_0207/10
- added R82: 68k, resistor:R-US_0207/10
- added TRIM11: 10k, rcl:R-TRIMM64W
- added TRIM12: 20 OHM, rcl:R-TRIMM64W
- C2: value 1nF -> 0.1uF
Connections:
- removed net CC_INPUT: C30.2, IC6.OUT, TRIM3.S
- removed net DRUM_OUTPUT: C27.1, IC5.OUT, R31.1, TRIM6.E
- removed net HIGH_FREQ_WN: C36.2, IC3.OUT, R11.1
- removed net LOW_FREQ_WN: C35.2, IC2.OUT, R10.1
- removed net N$1: R15.1, R17.1, R18.2
- removed net N$10: C35.1, R15.2
- removed net N$2: IC6.-IN, R35.1, R36.1, R38.2
- removed net N$27: IC3.-IN, R11.2, R7.1
- removed net N$3: R38.1, TRIM3.A
- removed net N$32: C2.1, IC3.+IN, R5.1
- removed net N$33: IC2.-IN, R10.2, R6.1
- removed net N$34: C4.1, IC2.+IN, R1.2
- removed net N$36: C20.2, C22.2, D2.C, R27.2
- removed net N$37: C30.1, Q6.B, R41.1, R42.2
- removed net N$38: C32.1, Q6.E, R44.2
- removed net N$39: C31.1, C33.+, Q6.C, R43.1
- removed net N$4: IC6.ON2, TRIM4.A
- removed net N$40: D2.A, Q4.E, R20.2
- removed net N$41: C22.1, IC5.+IN, R29.2
- removed net N$42: R23.2, TRIM1.S
- removed net N$43: C25.2, IC5.-IN, R31.2
- removed net N$45: IC5.ON1, TRIM5.E
- removed net N$46: IC5.ON2, TRIM5.A
- removed net N$48: IC4.+IN, R22.1, R28.2, TRIM1.A
- removed net N$49: IC4.-IN, Q5.D, R21.1, R30.2
- removed net N$50: IC4.ON1, TRIM2.E
- removed net N$51: C19.2, D1.C, R25.2
- removed net N$52: IC4.ON2, TRIM2.A
- removed net N$53: D1.A, Q3.E, R19.2
- removed net N$7: IC6.ON1, TRIM4.E
- removed net N$8: C25.1, C27.2, R32.2
- new net BRIDGED_T_OUT: C53.1, R75.1
- new net CC_INPUT1: C54.2
- new net FILTER_OUT: C2.2
- new net N$61: IC7.+IN, R64.1, R65.2
- new net N$62: C49.1, R65.1
- new net N$63: C54.1, Q17.B, R76.1, R77.2
- new net N$64: D3.A, Q15.E, R66.2
- new net N$65: IC8.+IN, R68.2, R71.1, TRIM12.A
- new net N$66: IC8.-IN, Q16.D, R69.2, R70.1
- new net N$67: IC8.ON2, TRIM11.A
- new net N$68: IC8.ON1, TRIM11.E
- new net N$69: R72.2, TRIM12.S
- new net N$70: R67.1, R73.2
- new net N$71: C56.1, Q17.E, R78.2
- new net N$72: C55.1, C57.+, Q17.C, R79.1
- new net N$73: C59.2, C60.1, R81.1
- new net N$74: C60.2, Q18.B, R82.1
- new net N$75: C2.1, Q18.E, R81.2, R83.1
- net +12V: now also C52.2, IC8.V+, Q15.C, Q18.C, R76.2, R79.2; no longer C11.2, C21.2, C23.1, C28.2, C9.2, IC2.V+, IC3.V+, IC4.V+, IC5.V+, IC6.V+, Q3.C, Q4.C, R41.2, R43.2
- net -12V: now also C51.2, IC8.V-, R77.1, R78.1, R83.2, TRIM11.S; no longer C10.2, C12.2, C24.2, C26.2, C29.2, IC2.V-, IC3.V-, IC4.V-, IC5.V-, IC6.V-, R42.1, R44.1, TRIM2.S, TRIM4.S, TRIM5.S
- net AGND: now also C50.1, C51.1, C52.1, C55.2, C57.-, C58.2, Q16.S, R64.2, R66.1, R68.1, R72.1, R73.1, R80.1, R82.2; no longer C10.1, C11.1, C12.1, C19.1, C20.1, C21.1, C23.2, C24.1, C26.1, C28.1, C29.1, C31.2, C33.-, C4.2, C9.1, IC6.+IN, IC7.+IN, Q5.S, R19.1, R20.1, R23.1, R26.1, R27.1, R28.1, R29.1, R32.1, R45.1, R5.2, R6.2, R7.2, TRIM6.A
- net N$60: now also C53.2
- net OUTPUT: now also C56.2, R80.2; no longer C32.2, R45.2
- net POT1A: no longer TRIM6.S
- net POT1B: no longer R35.2
- net POT2A: no longer C36.1
- net POT2B: no longer R17.2
- net SW1: now also C58.1, C59.1, IC8.OUT, R69.1; no longer IC4.OUT, R30.1
- net SW2: no longer R36.2
- net TRIGGER: now also Q15.B; no longer Q3.B, Q4.B
- net VCA_INPUT: now also R70.2, R71.2, R74.2, R75.2; no longer R18.1, R21.2, R22.2
- net VCA_TRIGGER: now also C50.2, D3.C, Q16.G, R67.2; no longer Q5.G, R25.1, R26.2
- net WHITE_NOISE_AMP: now also R74.1; no longer C2.2, R1.1
Other:
- note removed: "Drum Hit"
- note removed: "Extra Pins (In case I screwed something up)"
- note removed: "Note: 1) POT1A is the drum output 2) The third pin of POT1 should be grounded 3) POT1B should be the middle pin of the POT"
- note removed: "Note: 1) Switch turns the snare on/off 2) SW1 and SW2 normally connected 3) SW3 should be left open on the pot board"
- note removed: "Note: POT1B is the drum output"
- note removed: "Note: The third pin of POT2 should be grounded POT2B should be the middle pin"
- note removed: "Summing Amp and Common Collector"
- note removed: "Voltage-Controlled Amplifier"
- note removed: "WN High Pass Filter"
- note removed: "WN Low Pass Filter"
- moved on the sheet: C1, C13, C14, C15, C16, C17, C18, C2, C3, C34, C37, C38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

Commit message: Changed resistors out for shorter ones
changed resistors out for shorter ones
Parts:
- removed R54, R55: 20k, resistor:R-US_0207/10
- removed R56: 560, resistor:R-US_0207/10
- removed R57: 82k, resistor:R-US_0207/10
- removed R58, R59, R60, R61: 220k, resistor:R-US_0207/10
- removed R62, R67, R73, R80: 47k, resistor:R-US_0207/10
- removed R63, R64, R68, R69, R70, R71, R75, R76, R77, R78: 10k, resistor:R-US_0207/10
- removed R65, R83: 22k, resistor:R-US_0207/10
- removed R66: 470k, resistor:R-US_0207/10
- removed R72: 100, resistor:R-US_0207/10
- removed R74: 18k, resistor:R-US_0207/10
- removed R79: 220, resistor:R-US_0207/10
- removed R81: 2.7k, resistor:R-US_0207/10
- removed R82: 68k, resistor:R-US_0207/10
- added R1: 1k, rcl:R-US_0207/7
- added R10, R15, R18, R19, R22, R23, R31, R38, R41, R42: 10k, rcl:R-US_0207/7
- added R11, R17, R20, R21, R25: 20k, rcl:R-US_0207/7
- added R26, R30: 47k, rcl:R-US_0207/7
- added R27: 1 MEG, rcl:R-US_0207/7
- added R28, R7: 100k, rcl:R-US_0207/7
- added R29: 220k, rcl:R-US_0207/7
- added R32, R45: 22k, rcl:R-US_0207/7
- added R35: 560, rcl:R-US_0207/7
- added R36: 18k, rcl:R-US_0207/7
- added R43: 2.7k, rcl:R-US_0207/7
- added R44: 68k, rcl:R-US_0207/7
- added R5, R6: 2k, rcl:R-US_0207/7
- R12: value 4.7k -> 20k; device resistor:R-US_0207/10 -> rcl:R-US_0207/7
- R13: value 1k -> 10k; device resistor:R-US_0207/10 -> rcl:R-US_0207/7
- R14: value 100k -> 220k; device resistor:R-US_0207/10 -> rcl:R-US_0207/7
- R16: value 100k -> 20k; device resistor:R-US_0207/10 -> rcl:R-US_0207/7
- R2: value 47k -> 220k; device resistor:R-US_0207/10 -> rcl:R-US_0207/7
- R24: value 10k -> 20k; device resistor:R-US_0207/10 -> rcl:R-US_0207/7
- R3: value 2k -> 680k; device resistor:R-US_0207/10 -> rcl:R-US_0207/7
- R33, R39, R49, R52: device resistor:R-US_0207/10 -> rcl:R-US_0207/7
- R34: value 20k -> 82k; device resistor:R-US_0207/10 -> rcl:R-US_0207/7
- R37, R51: value 20k -> 10k; device resistor:R-US_0207/10 -> rcl:R-US_0207/7
- R4: value 2k -> 4.7k; device resistor:R-US_0207/10 -> rcl:R-US_0207/7
- R40: value 10k -> 100; device resistor:R-US_0207/10 -> rcl:R-US_0207/7
- R46: value 20k -> 27k; device resistor:R-US_0207/10 -> rcl:R-US_0207/7
- R47: value 20k -> 22k; device resistor:R-US_0207/10 -> rcl:R-US_0207/7
- R48: value 10k -> 470k; device resistor:R-US_0207/10 -> rcl:R-US_0207/7
- R50: value 20k -> 220; device resistor:R-US_0207/10 -> rcl:R-US_0207/7
- R53: value 10k -> 47k; device resistor:R-US_0207/10 -> rcl:R-US_0207/7
- R8: value 680k -> 10k; device resistor:R-US_0207/10 -> rcl:R-US_0207/7
- R9: value 1 MEG -> 220k; device resistor:R-US_0207/10 -> rcl:R-US_0207/7
Connections:
- removed net N$70: R67.1, R73.2
- new net N$1: C50.2, D3.C, R46.2
- net +12V: now also R10.2, R13.2, R15.2, R18.2, R19.2, R22.2, R23.2, R50.2, R52.2, R6.2, R8.2; no longer R24.1, R3.1, R33.1, R39.1, R40.1, R48.1, R49.1, R52.1, R53.1, R76.2, R79.2
- net -12V: now also R45.1, R49.1, R5.2, R51.1; no longer R4.2, R77.1, R78.1, R83.2
- net AGND: now also R28.2, R31.1, R33.1, R35.1, R40.1, R41.1, R44.1, R47.1, R48.1, R53.1; no longer R14.2, R56.2, R63.1, R64.2, R66.1, R68.1, R72.1, R73.1, R80.1, R82.2
- net BRIDGED_T_OUT: now also R37.1; no longer R75.1
- net N$11: now also R8.1; no longer R24.2
- net N$12: now also R11.1; no longer R34.2
- net N$13: now also R12.1; no longer R37.2
- net N$14: now also R34.1; no longer R57.1
- net N$15: now also R11.2, R12.2; no longer R34.1, R37.1
- net N$16: now also R15.1; no longer R39.2
- net N$18: now also R16.1; no longer R46.2
- net N$19: now also R17.1; no longer R47.2
- net N$20: now also R3.1; no longer R8.2
- net N$21: now also R1.1, R5.1, R7.1; no longer R13.2, R16.2, R4.1
- net N$22: now also R14.2, R2.2, R29.2, R30.1, R9.2; no longer R58.2, R59.2, R60.2, R61.2, R62.1
- net N$23: now also R26.1, R27.2; no longer R2.1, R9.2
- net N$28: now also R26.2; no longer R2.2
- net N$29: now also R16.2, R17.2; no longer R46.1, R47.1
- net N$30: now also R4.1; no longer R12.2
- net N$31: now also R18.1; no longer R48.2
- net N$35: now also R20.1; no longer R50.2
- net N$44: now also R21.1; no longer R51.2
- net N$47: now also R35.2; no longer R56.1
- net N$5: now also R1.2; no longer R13.1
- net N$54: now also R20.2, R21.2; no longer R50.1, R51.1
- net N$55: now also R22.1; no longer R52.2
- net N$56: now also R24.1; no longer R54.2
- net N$57: now also R25.1; no longer R55.2
- net N$58: now also R30.2, R31.2; no longer R62.2, R63.2
- net N$59: now also R24.2, R25.2; no longer R54.1, R55.1
- net N$6: now also R4.2, R6.1; no longer R12.1, R8.1
- net N$60: now also R34.2; no longer R57.2
- net N$61: now also R32.2, R33.2; no longer R64.1, R65.2
- net N$62: now also R32.1; no longer R65.1
- net N$63: now also R51.2, R52.1; no longer R76.1, R77.2
- net N$64: now also R48.2; no longer R66.2
- net N$65: now also R39.2, R41.2; no longer R68.2, R71.1
- net N$66: now also R38.2, R42.1; no longer R69.2, R70.1
- net N$69: now also R40.2; no longer R72.2
- net N$71: now also R49.2; no longer R78.2
- net N$72: now also R50.1; no longer R79.1
- net N$73: now also R43.2; no longer R81.1
- net N$74: now also R44.2; no longer R82.1
- net N$75: now also R43.1, R45.2; no longer R81.2, R83.1
- net N$9: now also R27.1; no longer R9.1
- net OSC1: now also R10.1, R2.1; no longer R33.2, R58.1
- net OSC2: now also R13.1, R9.1; no longer R40.2, R59.1
- net OSC3: now also R14.1, R19.1; no longer R49.2, R60.1
- net OSC4: now also R23.1, R29.1; no longer R53.2, R61.1
- net OUTPUT: now also R53.2; no longer R80.2
- net SW1: now also R42.2; no longer R69.1
- net VCA_INPUT: now also R36.2, R37.2, R38.1, R39.1; no longer R70.2, R71.2, R74.2, R75.2
- net VCA_TRIGGER: now also R46.1, R47.2; no longer C50.2, D3.C, R67.2
- net WHITE_NOISE: now also R7.2; no longer R16.1
- net WHITE_NOISE_AMP: now also R28.1, R36.1; no longer R14.1, R74.1
Other:
- moved on the sheet: R12, R13, R14, R16, R2, R24, R3, R33, R34, R37, R39, R4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

Commit message: Updates to cymbals
Parts:
- removed R36: 18k, rcl:R-US_0207/7
- removed R37: 10k, rcl:R-US_0207/7
- removed R40: 100, rcl:R-US_0207/7
- removed TRIM12: 20 OHM, rcl:R-TRIMM64W
- added C10, C11, C12, C4, C9: 0.1uF, resistor:C-EU050-024X044
- added IC2, IC3: LM741P, linear:LM741P
- added Q3, Q4, Q5: (no value), Capstone:J176
- added R54, R55, R57, R58, R59: 10k, rcl:R-US_0207/7
- added R56: 220k, rcl:R-US_0207/7
- added TRIM1: 10k, rcl:R-TRIMM64W
- R26: value 47k -> 68k
- R27: value 1 MEG -> 100k
Connections:
- removed net N$69: R40.2, TRIM12.S
- removed net VCA_INPUT: R36.2, R37.2, R38.1, R39.1
- new net N$10: IC3.OUT, R56.2
- new net N$2: IC2.+IN, Q4.D, R55.2, R57.2
- new net N$27: C12.1, R59.1
- new net N$3: IC2.-IN, Q3.D, R54.2, R58.1
- new net N$4: IC2.ON2, TRIM1.A
- new net N$7: IC2.ON1, TRIM1.E
- new net N$8: IC3.-IN, R56.1, R59.2
- new net SW4: C12.2, IC2.OUT, R58.2
- new net VCA_INPUT1: R54.1, R55.1
- net +12V: now also C11.2, C9.2, IC2.V+, IC3.V+
- net -12V: now also C10.2, C4.2, IC2.V-, IC3.V-, TRIM1.S
- net AGND: now also C10.1, C11.1, C4.1, C9.1, IC3.+IN, Q3.S, Q4.G, Q4.S, Q5.G, Q5.S, R57.1; no longer R40.1
- net BRIDGED_T_OUT: no longer R37.1
- net N$65: now also Q5.D; no longer TRIM12.A
- net VCA_TRIGGER: now also Q3.G
- net WHITE_NOISE_AMP: now also R38.1, R39.1; no longer R36.1

Commit message: Created Waveform generator board
Parts:
- removed C51, C52: 0.1uF, resistor:C-EU050-024X044
- removed C53: 22nF, resistor:C-EU050-024X044
- removed C54, C56: 2.2u, resistor:C-EU050-024X044
- removed C55: 1u, resistor:C-EU050-024X044
- removed C57: 10uF, rcl:CPOL-USE2.5-6
- removed C58: 1.5nF, resistor:C-EU050-024X044
- removed C59, C60: 1nF, resistor:C-EU050-024X044
- removed Q18: 2N3904, transistor:2N3904
- removed TRIM1, TRIM10, TRIM11, TRIM7, TRIM8, TRIM9: 10k, rcl:R-TRIMM64W
- added C19: 47nF, resistor:C-EU050-024X044
- added C20, C21: 33nF, resistor:C-EU050-024X044
- added C22: 0.47uF, resistor:C-EU050-024X044
- added C23: 1nF, resistor:C-EU050-024X044
- added C24, C27: 3.3nF, resistor:C-EU050-024X044
- added C25, C26, C29, C30, C31, C32, C33, C35, C36: 0.1uF, resistor:C-EU050-024X044
- added C28: 22nF, resistor:C-EU050-024X044
- added D1, D2, D4, D5: 200mA/100V/1V, SparkFun-DiscreteSemi:DIODE-1N4148
- added IC4, IC5, IC6: LM741P, linear:LM741P
- added Q6: 2N2222A, SparkFun-DiscreteSemi:TRANS_NPN-P2N2222A
- added R36: 220k, rcl:R-US_0207/7
- added R37, R69: 47k, rcl:R-US_0207/7
- added R40, R63, R65, R66, R68: 10k, rcl:R-US_0207/7
- added R60: 2.7k, rcl:R-US_0207/7
- added R61, R64: 68k, rcl:R-US_0207/7
- added R62: 22k, rcl:R-US_0207/7
- added R67: 220, rcl:R-US_0207/7
- C1, C2, C5, C8, C9: value 0.1uF -> 10uF; device resistor:C-EU050-024X044 -> rcl:CPOL-USE2.5-6
- C13, C14, C15, C16: value 10uF -> 0.1uF; device rcl:CPOL-USE2.5-6 -> resistor:C-EU050-024X044
- C17: value 1u -> 0.1uF
- C18: value 1u -> 47nF
- C3: value 10uF -> 1u; device rcl:CPOL-USE2.5-6 -> resistor:C-EU050-024X044
- C4: value 0.1uF -> 1u
- C41: value 47nF -> 1.5nF
- C42: value 47nF -> 1nF
- C43: value 33nF -> 1nF
- C44: value 33nF -> 0.1uF
- C47: value 3.3nF -> 2.2u
- C48: value 3.3nF -> 1u
- C49: value 1nF -> 2.2u
- C50: value 0.47uF -> 10uF; device resistor:C-EU050-024X044 -> rcl:CPOL-USE2.5-6
- Q1, Q2: value 2N3904 -> 2N2222A; device transistor:2N3904 -> SparkFun-DiscreteSemi:TRANS_NPN-P2N2222A
- Q10, Q11, Q12, Q13: value 2N2222A -> (none); device SparkFun-DiscreteSemi:TRANS_NPN-P2N2222A -> Capstone:J176
- Q14, Q15: value 2N2222A -> 2N3904; device SparkFun-DiscreteSemi:TRANS_NPN-P2N2222A -> transistor:2N3904
- Q16: value (none) -> 2N3904; device Capstone:J176 -> transistor:2N3904
- Q3, Q4, Q5: value (none) -> 2N2222A; device Capstone:J176 -> SparkFun-DiscreteSemi:TRANS_NPN-P2N2222A
- R1: value 1k -> 2k
- R12, R17: value 20k -> 10k; device rcl:R-US_0207/7 -> rcl:R-TRIMM64W
- R13, R18, R23: value 10k -> 20k
- R14, R29: value 220k -> 10k
- R2: value 220k -> 2k
- R20, R24, R25: value 20k -> 10k
- R22, R54: device rcl:R-US_0207/7 -> rcl:R-TRIMM64W
- R26: value 68k -> 20k
- R27: value 100k -> 10k; device rcl:R-US_0207/7 -> rcl:R-TRIMM64W
- R28: value 100k -> 20k
- R30: value 47k -> 470k
- R31: value 10k -> 27k
- R33: value 10k -> 220k
- R34: value 82k -> 220k
- R35: value 560 -> 220k
- R39: value 10k -> 22k
- R41: value 10k -> 82k
- R42: value 10k -> 560
- R43: value 2.7k -> 10k
- R44: value 68k -> 10k
- R45: value 22k -> 10k
- R46: value 27k -> 10k
- R47: value 22k -> 10k; device rcl:R-US_0207/7 -> rcl:R-TRIMM64W
- R48: value 470k -> 10k
- R49: value 10k -> 300k
- R5: value 2k -> 1k
- R50: value 220 -> 10k
- R53: value 47k -> 10k
- R57: value 10k -> 470k
- R58, R8: value 10k -> 100k
- R6: value 2k -> 100k
- R7: value 100k -> 68k
- R9: value 220k -> 100k
Connections:
- removed net CC_INPUT1: C54.2
- removed net VCA_INPUT1: R54.1, R55.1
- new net CYMBAL_PREFILTER: C41.1, C42.1, IC7.OUT, R59.2
- new net CYMBAL_SIGNAL: D4.C, D5.A, R57.1
- new net N$32: IC4.-IN, R48.2, R49.1
- new net N$33: IC8.-IN, R63.1, R64.2
- new net N$34: C31.1, R48.1
- new net N$36: C31.2, IC3.OUT, R46.2
- new net N$38: D2.A, D3.C, IC4.OUT, R49.2
- new net N$39: D4.A, D5.C, IC6.OUT, R56.2
- new net PRE_CC: C47.2, IC8.OUT, R64.1
- new net WN_SIGNAL: D2.C, D3.A, R58.1
- net +12V: now also C1.+, C25.2, C29.2, C3.2, C32.2, C34.2, C37.2, C39.2, C45.2, IC4.V+, IC5.V+, IC6.V+, Q16.C, Q9.C, R1.2, R12.E, R14.2, R17.E, R20.2, R22.E, R24.2, R25.2, R27.E, R29.2, R65.2, R67.2; no longer C15.+, C17.2, C46.2, C52.2, C7.2, C9.2, Q15.C, Q18.C, R13.2, R18.2, R22.2, R23.2, R50.2, R52.2, R6.2, R8.2, TRIM10.E, TRIM7.E, TRIM8.E, TRIM9.E
- net -12V: now also C12.2, C2.-, C26.2, C30.2, C33.2, C35.2, C38.2, C4.1, C40.2, C46.2, IC4.V-, IC5.V-, IC6.V-, R2.2, R47.S, R54.S, R62.1, R66.1, R68.1; no longer C10.2, C16.-, C18.1, C4.2, C45.2, C51.2, C8.2, R45.1, R49.1, R5.2, R51.1, TRIM1.S, TRIM11.S
- net AGND: now also C1.-, C12.1, C2.+, C22.1, C25.1, C26.1, C29.1, C3.1, C30.1, C32.1, C33.1, C34.1, C35.1, C37.1, C38.1, C39.1, C4.2, C40.1, C41.2, C48.2, C50.-, IC4.+IN, IC6.+IN, IC7.+IN, IC8.+IN, Q1.E, Q10.G, Q10.S, Q11.S, Q12.G, Q12.S, Q13.S, Q2.E, Q3.E, Q4.E, Q5.E, Q6.E, R30.1, R32.1, R38.1, R40.1, R42.1, R45.1, R52.1, R61.1, R69.1, R9.2; no longer C10.1, C15.-, C16.+, C17.1, C18.2, C4.1, C50.1, C51.1, C52.1, C55.2, C57.-, C58.2, C7.1, C8.1, C9.1, IC3.+IN, Q10.E, Q11.E, Q12.E, Q13.E, Q14.E, Q16.S, Q3.S, Q4.G, Q4.S, Q5.G, Q5.S, Q9.E, R28.2, R31.1, R33.1, R35.1, R41.1, R44.1, R47.1, R48.1, R53.1, R57.1
- net BRIDGED_T_OUT: now also C28.1, R50.1, R51.1; no longer C53.1
- net FILTER_OUT: now also C44.2, R63.2; no longer C2.2
- net N$1: now also C22.2, D1.C, R31.2; no longer C50.2, D3.C, R46.2
- net N$10: now also IC7.-IN, R57.2, R58.2, R59.1; no longer IC3.OUT, R56.2
- net N$11: now also C14.2, Q1.C, R10.1; no longer C37.2, Q8.C, R8.1
- net N$12: now also C14.1, Q2.B; no longer C37.1, Q7.B
- net N$13: now also C15.2, Q1.B, R13.1; no longer C38.2, Q8.B, R12.1
- net N$14: now also C24.2, IC2.-IN, R41.1; no longer C47.2, IC7.-IN, R34.1
- net N$15: now also R12.S, R13.2; no longer R12.2, TRIM7.S
- net N$16: now also C16.2, Q3.C; no longer C39.2, Q10.C
- net N$17: now also Q14.B, Q15.B; no longer Q1.B, Q2.B
- net N$18: now also C16.1, Q4.B; no longer C39.1, Q9.B
- net N$19: now also C17.2, Q3.B, R18.1; no longer C40.2, Q10.B, R17.1
- net N$2: now also IC5.+IN, Q12.D, R51.2, R52.2; no longer IC2.+IN, Q4.D, R55.2, R57.2
- net N$20: now also C7.1, Q14.E; no longer C6.1, Q1.E
- net N$21: now also C5.-, C6.1, C9.-, R2.1, R6.1; no longer C14.-, C3.-, C5.1, R1.1, R7.1
- net N$22: now also R33.2, R34.2, R35.2, R36.2, R37.1; no longer R14.2, R2.2, R29.2, R30.1, R9.2
- net N$23: now also R7.1, R8.2; no longer R26.1, R27.2
- net N$27: now also C36.1, R55.1; no longer C12.1, R59.1
- net N$28: now also C10.1, R7.2; no longer C1.1, R26.2
- net N$29: now also R17.S, R18.2; no longer R17.2, TRIM8.S
- net N$3: now also IC5.-IN, Q13.D, R50.2, R53.1; no longer IC2.-IN, Q3.D, R54.2, R58.1
- net N$30: now also C8.+, Q15.C; no longer C13.+, Q2.C
- net N$31: now also C18.2, Q5.C, R20.1; no longer C41.2, Q12.C, R18.1
- net N$35: now also C18.1, Q6.B, R21.1; no longer C41.1, Q11.B, R20.1
- net N$4: now also IC5.ON2, R54.A; no longer IC2.ON2, TRIM1.A
- net N$44: now also C19.2, Q5.B, R23.1; no longer C42.2, Q12.B, R21.1
- net N$47: now also C24.1, C27.2, R42.2; no longer C47.1, C48.2, R35.2
- net N$5: now also C9.+, Q15.E, R5.2; no longer C14.+, Q2.E, R1.2
- net N$54: now also R22.S, R23.2; no longer R20.2, TRIM9.S
- net N$55: now also C20.2, Q7.C, R25.1; no longer C43.2, Q14.C, R22.1
- net N$56: now also C20.1, Q8.B, R26.1; no longer C43.1, Q13.B, R24.1
- net N$57: now also C21.2, Q7.B, R28.1; no longer C44.2, Q14.B, R25.1
- net N$58: now also C23.2, R37.2, R38.2; no longer C49.2, R30.2, R31.2
- net N$59: now also R26.2, R27.S, R28.2; no longer R24.2, R25.2, TRIM10.S
- net N$6: now also C5.+, C7.2, R1.1; no longer C3.+, C5.2, R6.1
- net N$60: now also C27.1, C28.2, IC2.OUT, R41.2; no longer C48.1, C53.2, IC7.OUT, R34.2
- net N$61: now also IC2.+IN, R39.2, R40.2; no longer IC7.+IN, R32.2, R33.2
- net N$62: now also C23.1, R39.1; no longer C49.1, R32.1
- net N$63: now also C47.1, R65.1, R66.2; no longer C54.1, R51.2, R52.1
- net N$64: now also D1.A, Q9.E, R30.2; no longer D3.A, Q15.E, R48.2
- net N$65: now also IC3.+IN, Q10.D, R44.2, R45.2; no longer IC8.+IN, Q5.D, R39.2, R41.2
- net N$66: now also IC3.-IN, Q11.D, R43.2, R46.1; no longer IC8.-IN, Q16.D, R38.2, R42.1
- net N$67: now also IC3.ON2, R47.A; no longer IC8.ON2, TRIM11.A
- net N$68: now also IC3.ON1, R47.E; no longer IC8.ON1, TRIM11.E
- net N$7: now also IC5.ON1, R54.E; no longer IC2.ON1, TRIM1.E
- net N$71: now also C49.1, R68.2; no longer C56.1, R49.2
- net N$72: now also C48.1, C50.+, R67.1; no longer C55.1, C57.+, R50.1
- net N$73: now also C42.2, C43.1, R60.2; no longer C59.2, C60.1, R43.2
- net N$74: now also C43.2, Q16.B, R61.2; no longer C60.2, Q18.B, R44.2
- net N$75: now also C44.1, Q16.E, R60.1, R62.2; no longer C2.1, Q18.E, R43.1, R45.2
- net N$8: now also IC6.-IN, R55.2; no longer IC3.-IN, R59.2
- net N$9: now also C13.2, R8.1; no longer C34.2, R27.1
- net OSC1: now also C15.1, Q2.C, R14.1, R33.1; no longer C38.1, Q7.C, R10.1, R2.1
- net OSC2: now also C17.1, Q4.C, R19.1, R34.1; no longer C40.1, Q9.C, R13.1, R9.1
- net OSC3: now also C19.1, Q6.C, R24.1, R35.1; no longer C42.1, Q11.C, R14.1, R19.1
- net OSC4: now also C21.1, Q8.C, R36.1; no longer C44.1, Q13.C, R23.1
- net OUTPUT: now also C49.2, R69.2; no longer C56.2, R53.2
- net SW1: no longer C58.1, C59.1, IC8.OUT, R42.2
- net SW4: now also C36.2, IC5.OUT, R53.2; no longer C12.2, IC2.OUT, R58.2
- net TRIGGER: now also Q9.B; no longer Q15.B
- net VCA_TRIGGER: now also Q11.G, Q13.G, R31.1, R32.2; no longer Q16.G, Q3.G, R46.1, R47.2
- net WHITE_NOISE: now also C10.2, C8.-, R6.2; no longer C1.2, C13.-, R7.2
- net WHITE_NOISE_AMP: now also C13.1, R43.1, R44.1, R9.1; no longer C34.1, R28.1, R38.1, R39.1
Other:
- moved on the sheet: C10, C11, C12, C17, C18, C34, C37, C38, C39, C4, C40, C41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
