File: Hi Hat/PCB/Hi-Hat.sch (EAGLE design)
At the start: 92 parts, among them IC1 LM741P, IC2 LM741P, IC3 LM741P, IC4 LM741P, IC5 LM741P, IC6 LM741P, IC7 LM741P, Q1 2N2222A, Q6 2N3904, Q7 2N3904

Commit message: Added text
Other:
- note added: "Note: used 330k"
- note added: "used 2.2k"
Changed lines of the file:
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@@
 <text x="1620.52" y="388.62" size="1.778" layer="94">Note: Resistor at the collector should be a jumper.
 The resistor is only there so biasing can be changed if needed.</text>
+<text x="1280.16" y="388.62" size="1.778" layer="91">Note: used 330k</text>
+<text x="1605.28" y="350.52" size="1.778" layer="91">used 2.2k</text>
 </plain>
 <instances>

Commit message: Cleaned up schematics
Other:
- note added: "24 Pin Header"
- note added: "Bridged-T Oscillator"
- note added: "Common Collector Output"
- note added: "Cymbal VCA"
- note added: "Cymbal VCA Amplifier"
- note added: "Envelope Generator"
- note added: "Filter"
- note added: "Summing Stage"
- note added: "Waveform Generator Input"
- note added: "White Noise VCA"
- note added: "White Noise VCA Amplifier"
- moved on the sheet: C1, C10, C11, C12, C13, C14, C15, C16, C17, C18, C19, C2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
