File: Hi Hat/PCB/Cymbal Waveform Generator Board.sch (EAGLE design)
At the start: 92 parts, among them IC1 LM741P, IC2 LM741P, IC3 LM741P, IC4 LM741P, IC5 LM741P, IC6 LM741P, IC7 LM741P, Q1 2N2222A, Q2 J176, Q3 J176, Q4 J176, Q5 J176, Q6 2N3904, Q7 2N3904

Commit message: Updated cymbal schematics
Parts:
- removed C29, C30: 0.1uF, resistor:C-EU050-024X044
- removed C31, C33: 2.2u, resistor:C-EU050-024X044
- removed C32: 1u, resistor:C-EU050-024X044
- removed C34: 10uF, rcl:CPOL-USE2.5-6
- removed D1, D2, D3, D4, D5: 200mA/100V/1V, SparkFun-DiscreteSemi:DIODE-1N4148
- removed IC2, IC3, IC4, IC5, IC6, IC7: LM741P, linear:LM741P
- removed R16, R31: 10k, rcl:R-US_0207/7
- removed R21: 300k, rcl:R-US_0207/7
- removed R26: 68k, rcl:R-US_0207/7
- added 1136_HZ, 305_HZ, 444_HZ, 794_HZ: (no value), SparkFun-Connectors:CONN_01PTH_NO_SILK_KIT
- added J3, J4, J5, J6: (no value), SparkFun-Connectors:CONN_031X03_NO_SILK
- added J7, J8: (no value), SparkFun-Connectors:CONN_021X02_NO_SILK
- added Q10, Q11, Q12, Q9: 2N3904, transistor:2N3904
- added Q8: 2N2222A, SparkFun-DiscreteSemi:TRANS_NPN-P2N2222A
- added R19, R39, R40, R41, R43: 10k, rcl:R-US_0207/7
- added R36, R37: 220k, rcl:R-US_0207/7
- added R38, R44: 47k, rcl:R-US_0207/7
- added R42: 220, rcl:R-US_0207/7
- added TRIM3, TRIM4: 10k, Capstone:10K_TRIMMER
- C10: value 22nF -> 0.1uF
- C11: value 0.47uF -> 0.1uF
- C12: value 10uF -> 0.1uF; device rcl:CPOL-USE2.5-6 -> resistor:C-EU050-024X044
- C13, C15: value 0.1uF -> 2.2u
- C14: value 0.1uF -> 1u
- C16, C28, C8: value 0.1uF -> 10uF; device resistor:C-EU050-024X044 -> rcl:CPOL-USE2.5-6
- C21, C22: value 0.1uF -> 47nF
- C23, C24: value 0.1uF -> 33nF
- C25: value 1.5nF -> 2.2u
- C26: value 1nF -> 1u
- C27: value 1nF -> 2.2u
- C5: value 1nF -> 10uF; device resistor:C-EU050-024X044 -> rcl:CPOL-USE2.5-6
- C6: value 3.3nF -> 0.1uF
- C9: value 3.3nF -> 10uF; device resistor:C-EU050-024X044 -> rcl:CPOL-USE2.5-6
- J2: device SparkFun-Connectors:CONN_02 -> SparkFun-Connectors:CONN_031X03_NO_SILK
- Q2, Q3, Q4, Q5: value J176 -> 2N2222A; device Capstone:J176 -> SparkFun-DiscreteSemi:TRANS_NPN-P2N2222A
- Q6, Q7: value 2N3904 -> 2N2222A; device transistor:2N3904 -> SparkFun-DiscreteSemi:TRANS_NPN-P2N2222A
- R1: value 22k -> 2k
- R11: value 10k -> 220
- R12, R28: value 22k -> 10k
- R13: value 10k -> 47k
- R14: value 220k -> 10k
- R15, R17, R20, R32: value 10k -> 20k
- R2: value 10k -> 2k
- R22: value 470k -> 20k
- R23: value 100k -> 10k
- R25: value 2.7k -> 20k
- R27: value 0 -> 20k
- R3: value 82k -> 680k
- R30: value 68k -> 20k
- R33: value 220 -> 10k
- R34: value 10k -> 220k
- R35: value 47k -> 220k
- R4: value 560 -> 4.7k
- R5: value 470k -> 1k
- R6: value 27k -> 100k
- R7: value 22k -> 68k
- R8: value 10k -> 100k
Connections:
- removed net BRIDGED_T_OUT: C10.1, R8.1, R9.1
- removed net CYMBAL_PREFILTER: C25.1, C26.1, IC6.OUT, R24.2
- removed net CYMBAL_SIGNAL: D2.C, D3.A, R22.1
- removed net FILTER_OUT: C28.2, R29.2
- removed net N$1: C15.2, IC2.OUT, R11.2
- removed net N$10: IC6.-IN, R22.2, R23.2, R24.1
- removed net N$14: C6.2, IC1.-IN, R3.1
- removed net N$27: C15.1, R13.1
- removed net N$32: IC5.-IN, R20.2, R21.1
- removed net N$33: IC7.-IN, R29.1, R30.2
- removed net N$34: C20.1, R20.1
- removed net N$36: C20.2, IC4.OUT, R18.2
- removed net N$38: D4.A, D5.C, IC5.OUT, R21.2
- removed net N$39: D2.A, D3.C, IC3.OUT, R14.2
- removed net N$47: C6.1, C9.2, R4.2
- removed net N$60: C10.2, C9.1, IC1.OUT, R3.2
- removed net N$61: IC1.+IN, R1.2, R2.2
- removed net N$62: C5.1, R1.1
- removed net N$64: D1.A, Q1.E, R5.2
- removed net N$65: IC4.+IN, Q4.D, R16.2, R17.2
- removed net N$66: IC4.-IN, Q5.D, R15.2, R18.1
- removed net N$67: IC4.ON2, TRIM2.A
- removed net N$68: IC4.ON1, TRIM2.E
- removed net N$7: IC2.ON1, TRIM1.E
- removed net N$73: C26.2, C27.1, R25.2
- removed net N$74: C27.2, Q6.B, R26.2
- removed net N$75: C28.1, Q6.E, R25.1, R28.2
- removed net N$8: IC3.-IN, R13.2, R14.1
- removed net PRE_CC: C31.2, IC7.OUT, R30.1
- removed net SQ_BUFFERED: C5.2, J1.2, J1.4, J1.6
- removed net VCA_TRIGGER: Q3.G, Q5.G, R6.1, R7.2
- removed net WN_BUFFERED: J1.1, J1.3, J1.5, R15.1, R16.1
- new net N$11: C17.2, Q1.C, R14.1
- new net N$12: C17.1, Q2.B, R15.1
- new net N$13: C18.2, Q1.B, R17.1
- new net N$15: R15.2, R17.2, TRIM1.S
- new net N$16: C19.2, Q3.C, R19.1
- new net N$17: Q10.B, Q11.B
- new net N$18: C19.1, Q4.B, R20.1
- new net N$19: C20.2, Q3.B, R22.1
- new net N$20: C7.1, Q10.E, R3.1
- new net N$21: C5.-, C6.1, C9.-, R2.1, R5.1, R6.1
- new net N$22: R34.2, R35.2, R36.2, R37.2, R38.1
- new net N$23: IC1.-IN, R7.1, R8.2
- new net N$28: C10.1, R7.2
- new net N$29: R20.2, R22.2, TRIM2.S
- new net N$30: C8.+, Q11.C, R4.1
- new net N$31: C21.2, Q5.C, R24.1
- new net N$35: C21.1, Q6.B, R25.1
- new net N$44: C22.2, Q5.B, R27.1
- new net N$54: R25.2, R27.2, TRIM3.S
- new net N$55: C23.2, Q7.C, R29.1
- new net N$56: C23.1, Q8.B, R30.1
- new net N$57: C24.2, Q7.B, R32.1
- new net N$58: C25.2, R38.2, R39.2
- new net N$59: R30.2, R32.2, TRIM4.S
- new net N$9: C13.2, IC1.OUT, R8.1
- new net OSC1: 305_HZ.1, C18.1, Q2.C, R18.1, R34.1
- new net OSC2: 444_HZ.1, C20.1, Q4.C, R23.1, R35.1
- new net OSC3: 794_HZ.1, C22.1, Q6.C, R28.1, R36.1
- new net OSC4: 1136_HZ.1, C24.1, Q8.C, R33.1, R37.1
- new net POT2B: SV1.7
- new net SQUARE_WAVE_BUFFERED: C27.2, J1.2, J1.4, J1.6, R44.2
- new net WHITE_NOISE: C10.2, C8.-, R6.2
- new net WHITE_NOISE_BUFFERED: C15.2, J1.1, J1.3, J1.5, R13.2
- net +12V: now also C11.2, R1.2, R11.2, R14.2, R18.2, R19.2, R23.2, R24.2, R28.2, R29.2, R40.2, R42.2, R9.2, TRIM1.E, TRIM2.E, TRIM3.E, TRIM4.E; no longer C13.2, C16.2, C18.2, C21.2, C23.2, C29.2, C7.2, IC2.V+, IC3.V+, IC4.V+, IC5.V+, IC6.V+, IC7.V+, Q1.C, R27.1, R31.2
- net -12V: now also C12.2, R10.1, R12.1, R2.2, R41.1, R43.1; no longer C14.2, C17.2, C19.2, C22.2, C24.2, C30.2, C8.2, IC2.V-, IC3.V-, IC4.V-, IC5.V-, IC6.V-, IC7.V-, R28.1, R32.1, R34.1, TRIM1.S, TRIM2.S
- net AGND: now also C12.1, C14.2, C16.-, C26.2, C28.-, IC1.+IN, Q1.E, Q2.E, Q3.E, Q4.E, Q5.E, Q6.E, Q7.E, Q8.E, R13.1, R39.1, R44.1; no longer C12.-, C13.1, C14.1, C16.1, C17.1, C18.1, C19.1, C21.1, C22.1, C23.1, C24.1, C25.2, C29.1, C30.1, C32.2, C34.-, C7.1, C8.1, IC3.+IN, IC5.+IN, IC6.+IN, IC7.+IN, Q2.G, Q2.S, Q3.S, Q4.G, Q4.S, Q5.S, R10.1, R17.1, R2.1, R26.1, R35.1, R4.1, R5.1, R7.1, SV1.7
- net N$2: now also C13.1, Q12.B, R9.1; no longer IC2.+IN, Q2.D, R9.2
- net N$3: now also C15.1, Q12.E, R12.2; no longer IC2.-IN, Q3.D, R11.1, R8.2
- net N$4: now also C14.1, C16.+, Q12.C, R11.1; no longer IC2.ON2, TRIM1.A
- net N$5: now also C9.+, Q11.E, R5.2; no longer Q6.C, R27.2
- net N$6: now also C5.+, C6.2, C7.2, R1.1, R3.2, R4.2; no longer C11.2, C12.+, D1.C, R12.2, R6.2
- net N$63: now also C25.1, Q9.B, R40.1, R41.2; no longer C31.1, Q7.B, R31.1, R32.2
- net N$71: now also C27.1, Q9.E, R43.2; no longer C33.1, Q7.E, R34.2
- net N$72: now also C26.1, C28.+, Q9.C, R42.1; no longer C32.1, C34.+, Q7.C, R33.1
- net OUTPUT: no longer C33.2, R35.2
- net POT1A: no longer D4.C, D5.A, J2.1
- net POT1B: no longer J2.2, R23.1
- net POT2A: no longer R12.1
- net TRIGGER: no longer Q1.B
Other:
- note added: "1136 Hz Oscillator Trimpot should be around 2.19k"
- note added: "305 Hz Oscillator Trimpot should be around 3.91k"
- note added: "444 Hz Oscillator Trimpot should be around 550 ohms"
- note added: "794 Hz Oscillator Trimpot should be around 2.05k"
- note added: "Output to Cymbals"
- note added: "Square Wave Buffer"
- note added: "Square Wave Generators"
- note added: "White Noise Amplifier / Buffer"
- note added: "White Noise Generator"
- note removed: "Bridged-T Oscillator"
- note removed: "Common Collector Output"
- note removed: "Cymbal VCA"
- note removed: "Cymbal VCA Amplifier"
- note removed: "Envelope Generator"
- note removed: "Filter"
- note removed: "Note: POT2B is grounded to AGND"
- note removed: "Note: R27 should be a jumper. The resistor is only there so biasing can be changed if needed."
- note removed: "Note: Short Jumper for open hi-hat Third pin of POT1 should be grounded"
- note removed: "Note: used 330k"
- note removed: "Summing Stage"
- note removed: "Waveform Generator Input"
- note removed: "White Noise VCA"
- note removed: "White Noise VCA Amplifier"
- note removed: "used 2.2k"
- moved on the sheet: C1, C10, C11, C13, C14, C15, C17, C18, C19, C2, C20, C21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
