File: Hi Hat/PCB/Cymbals.sch (EAGLE design)
At the start: 95 parts, among them IC1 LM741P, Q1 2N2222A, Q10 2N3904, Q11 2N3904, Q12 2N3904, Q2 2N2222A, Q3 2N2222A, Q4 2N2222A, Q5 2N2222A, Q6 2N2222A, Q7 2N2222A, Q8 2N2222A, Q9 2N3904

Commit message: Cleaned up schematics
Parts:
- removed J3, J4, J5, J6: (no value), SparkFun-Connectors:CONN_031X03_NO_SILK
- removed J7, J8: (no value), SparkFun-Connectors:CONN_021X02_NO_SILK
- removed J9: (no value), SparkFun-Connectors:CONN_041X04_NO_SILK
- removed Q10, Q11, Q12, Q9: 2N3904, transistor:2N3904
- removed Q8: 2N2222A, SparkFun-DiscreteSemi:TRANS_NPN-P2N2222A
- removed R19, R39, R40, R41, R43: 10k, rcl:R-US_0207/7
- removed R36, R37: 220k, rcl:R-US_0207/7
- removed R38, R44: 47k, rcl:R-US_0207/7
- removed R42: 220, rcl:R-US_0207/7
- removed TRIM3, TRIM4: 10k, Capstone:10K_TRIMMER
- added C29, C30: 0.1uF, resistor:C-EU050-024X044
- added C31, C33: 2.2u, resistor:C-EU050-024X044
- added C32: 1u, resistor:C-EU050-024X044
- added C34: 10uF, rcl:CPOL-USE2.5-6
- added D1, D2, D3, D4, D5: 200mA/100V/1V, SparkFun-DiscreteSemi:DIODE-1N4148
- added IC2, IC3, IC4, IC5, IC6, IC7: LM741P, linear:LM741P
- added R16, R31: 10k, rcl:R-US_0207/7
- added R21: 300k, rcl:R-US_0207/7
- added R26: 68k, rcl:R-US_0207/7
- C10: value 0.1uF -> 22nF
- C11: value 0.1uF -> 0.47uF
- C12: value 0.1uF -> 10uF; device resistor:C-EU050-024X044 -> rcl:CPOL-USE2.5-6
- C13, C15: value 2.2u -> 0.1uF
- C14: value 1u -> 0.1uF
- C16, C28, C8: value 10uF -> 0.1uF; device rcl:CPOL-USE2.5-6 -> resistor:C-EU050-024X044
- C21, C22: value 47nF -> 0.1uF
- C23, C24: value 33nF -> 0.1uF
- C25: value 2.2u -> 1.5nF
- C26: value 1u -> 1nF
- C27: value 2.2u -> 1nF
- C5: value 10uF -> 1nF; device rcl:CPOL-USE2.5-6 -> resistor:C-EU050-024X044
- C6: value 0.1uF -> 3.3nF
- C9: value 10uF -> 3.3nF; device rcl:CPOL-USE2.5-6 -> resistor:C-EU050-024X044
- J2: device SparkFun-Connectors:CONN_031X03_NO_SILK -> SparkFun-Connectors:CONN_02
- Q2, Q3, Q4, Q5: value 2N2222A -> J176; device SparkFun-DiscreteSemi:TRANS_NPN-P2N2222A -> Capstone:J176
- Q6, Q7: value 2N2222A -> 2N3904; device SparkFun-DiscreteSemi:TRANS_NPN-P2N2222A -> transistor:2N3904
- R1: value 2k -> 22k
- R11: value 220 -> 10k
- R12, R28: value 10k -> 22k
- R13: value 47k -> 10k
- R14: value 10k -> 220k
- R15, R17, R20, R32: value 20k -> 10k
- R2: value 2k -> 10k
- R22: value 20k -> 470k
- R23: value 10k -> 100k
- R25: value 20k -> 2.7k
- R27: value 20k -> 0
- R3: value 680k -> 82k
- R30: value 20k -> 68k
- R33: value 10k -> 220
- R34: value 220k -> 10k
- R35: value 220k -> 47k
- R4: value 4.7k -> 560
- R5: value 1k -> 470k
- R6: value 100k -> 27k
- R7: value 68k -> 22k
- R8: value 100k -> 10k
Connections:
- removed net N$11: C17.2, Q1.C, R14.1
- removed net N$12: C17.1, Q2.B, R15.1
- removed net N$13: C18.2, Q1.B, R17.1
- removed net N$15: R15.2, R17.2, TRIM1.S
- removed net N$16: C19.2, Q3.C, R19.1
- removed net N$17: Q10.B, Q11.B
- removed net N$18: C19.1, Q4.B, R20.1
- removed net N$19: C20.2, Q3.B, R22.1
- removed net N$20: C7.1, Q10.E, R3.1
- removed net N$21: C5.-, C6.1, C9.-, R2.1, R5.1, R6.1
- removed net N$22: R34.2, R35.2, R36.2, R37.2, R38.1
- removed net N$23: IC1.-IN, R7.1, R8.2
- removed net N$28: C10.1, R7.2
- removed net N$29: R20.2, R22.2, TRIM2.S
- removed net N$30: C8.+, Q11.C, R4.1
- removed net N$31: C21.2, Q5.C, R24.1
- removed net N$35: C21.1, Q6.B, R25.1
- removed net N$44: C22.2, Q5.B, R27.1
- removed net N$54: R25.2, R27.2, TRIM3.S
- removed net N$55: C23.2, Q7.C, R29.1
- removed net N$56: C23.1, Q8.B, R30.1
- removed net N$57: C24.2, Q7.B, R32.1
- removed net N$58: C25.2, R38.2, R39.2
- removed net N$59: R30.2, R32.2, TRIM4.S
- removed net N$9: C13.2, IC1.OUT, R8.1
- removed net OSC1: C18.1, Q2.C, R18.1, R34.1
- removed net OSC2: C20.1, Q4.C, R23.1, R35.1
- removed net OSC3: C22.1, Q6.C, R28.1, R36.1
- removed net OSC4: C24.1, Q8.C, R33.1, R37.1
- removed net POT2B: SV1.7
- removed net SQUARE_WAVE_BUFFERED: C27.2, J1.2, J1.4, J1.6, R44.2
- removed net WHITE_NOISE: C10.2, C8.-, R6.2
- removed net WHITE_NOISE_BUFFERED: C15.2, J1.1, J1.3, J1.5, R13.2
- new net BRIDGED_T_OUT: C10.1, R8.1, R9.1
- new net CYMBAL_PREFILTER: C25.1, C26.1, IC6.OUT, R24.2
- new net CYMBAL_SIGNAL: D2.C, D3.A, R22.1
- new net FILTER_OUT: C28.2, R29.2
- new net N$14: C6.2, IC1.-IN, R3.1
- new net N$27: C15.1, R13.1
- new net N$32: IC5.-IN, R20.2, R21.1
- new net N$33: IC7.-IN, R29.1, R30.2
- new net N$34: C20.1, R20.1
- new net N$36: C20.2, IC4.OUT, R18.2
- new net N$38: D4.A, D5.C, IC5.OUT, R21.2
- new net N$39: D2.A, D3.C, IC3.OUT, R14.2
- new net N$47: C6.1, C9.2, R4.2
- new net N$60: C10.2, C9.1, IC1.OUT, R3.2
- new net N$61: IC1.+IN, R1.2, R2.2
- new net N$62: C5.1, R1.1
- new net N$64: D1.A, Q1.E, R5.2
- new net N$65: IC4.+IN, Q4.D, R16.2, R17.2
- new net N$66: IC4.-IN, Q5.D, R15.2, R18.1
- new net N$67: IC4.ON2, TRIM2.A
- new net N$68: IC4.ON1, TRIM2.E
- new net N$73: C26.2, C27.1, R25.2
- new net N$74: C27.2, Q6.B, R26.2
- new net N$75: C28.1, Q6.E, R25.1, R28.2
- new net PRE_CC: C31.2, IC7.OUT, R30.1
- new net SQ_BUFFERED: C5.2, J1.2, J1.4, J1.6
- new net VCA_TRIGGER: Q3.G, Q5.G, R6.1, R7.2
- new net WN_BUFFERED: J1.1, J1.3, J1.5, R15.1, R16.1
- net +12V: now also C13.2, C16.2, C18.2, C21.2, C23.2, C29.2, C7.2, IC2.V+, IC3.V+, IC4.V+, IC5.V+, IC6.V+, IC7.V+, Q1.C, R27.1, R31.2; no longer C11.2, R1.2, R11.2, R14.2, R18.2, R19.2, R23.2, R24.2, R28.2, R29.2, R40.2, R42.2, R9.2, TRIM1.E, TRIM2.E, TRIM3.E, TRIM4.E
- net -12V: now also C14.2, C17.2, C19.2, C22.2, C24.2, C30.2, C8.2, IC2.V-, IC3.V-, IC4.V-, IC5.V-, IC6.V-, IC7.V-, R28.1, R32.1, R34.1, TRIM1.S, TRIM2.S; no longer C12.2, R10.1, R12.1, R2.2, R41.1, R43.1
- net AGND: now also C12.-, C13.1, C14.1, C16.1, C17.1, C18.1, C19.1, C21.1, C22.1, C23.1, C24.1, C25.2, C29.1, C30.1, C32.2, C34.-, C7.1, C8.1, IC3.+IN, IC5.+IN, IC6.+IN, IC7.+IN, Q2.G, Q2.S, Q3.S, Q4.G, Q4.S, Q5.S, R10.1, R17.1, R2.1, R26.1, R35.1, R4.1, R5.1, R7.1, SV1.7; no longer C12.1, C14.2, C16.-, C26.2, C28.-, IC1.+IN, Q1.E, Q2.E, Q3.E, Q4.E, Q5.E, Q6.E, Q7.E, Q8.E, R13.1, R39.1, R44.1
- net N$1: now also C15.2, IC2.OUT, R11.2; no longer J9.1
- net N$10: now also IC6.-IN, R22.2, R23.2, R24.1; no longer J9.4
- net N$2: now also IC2.+IN, Q2.D, R9.2; no longer C13.1, Q12.B, R9.1
- net N$3: now also IC2.-IN, Q3.D, R11.1, R8.2; no longer C15.1, Q12.E, R12.2
- net N$4: now also IC2.ON2, TRIM1.A; no longer C14.1, C16.+, Q12.C, R11.1
- net N$5: now also Q6.C, R27.2; no longer C9.+, Q11.E, R5.2
- net N$6: now also C11.2, C12.+, D1.C, R12.2, R6.2; no longer C5.+, C6.2, C7.2, R1.1, R3.2, R4.2
- net N$63: now also C31.1, Q7.B, R31.1, R32.2; no longer C25.1, Q9.B, R40.1, R41.2
- net N$7: now also IC2.ON1, TRIM1.E; no longer J9.2
- net N$71: now also C33.1, Q7.E, R34.2; no longer C27.1, Q9.E, R43.2
- net N$72: now also C32.1, C34.+, Q7.C, R33.1; no longer C26.1, C28.+, Q9.C, R42.1
- net N$8: now also IC3.-IN, R13.2, R14.1; no longer J9.3
- net OUTPUT: now also C33.2, R35.2
- net POT1A: now also D4.C, D5.A, J2.1
- net POT1B: now also J2.2, R23.1
- net POT2A: now also R12.1
- net TRIGGER: now also Q1.B
Other:
- note added: "24 Pin Header"
- note added: "Bridged-T Oscillator"
- note added: "Common Collector Output"
- note added: "Cymbal VCA"
- note added: "Cymbal VCA Amplifier"
- note added: "Envelope Generator"
- note added: "Filter"
- note added: "Note: POT2B is grounded to AGND"
- note added: "Note: R27 should be a jumper. The resistor is only there so biasing can be changed if needed."
- note added: "Note: Short Jumper for open hi-hat Third pin of POT1 should be grounded"
- note added: "Note: used 330k"
- note added: "Summing Stage"
- note added: "Waveform Generator Input"
- note added: "White Noise VCA"
- note added: "White Noise VCA Amplifier"
- note added: "used 2.2k"
- note removed: "1136 Hz Oscillator Trimpot should be around 2.19k"
- note removed: "305 Hz Oscillator Trimpot should be around 3.91k"
- note removed: "444 Hz Oscillator Trimpot should be around 550 ohms"
- note removed: "794 Hz Oscillator Trimpot should be around 2.05k"
- note removed: "White Noise Amplifier / Buffer"
- note removed: "White Noise Generator"
- moved on the sheet: C1, C10, C11, C13, C14, C15, C17, C18, C19, C2, C20, C21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

Commit message: Updated cymbal schematics
Other:
- note added: "Note: 1) Short Jumper for open hi-hat 2) Third pin of POT1 should be grounded"
- note added: "Note: used 2.2k since 2.7k was not available"
- note removed: "Note: Short Jumper for open hi-hat Third pin of POT1 should be grounded"
- note removed: "used 2.2k"
Changed lines of the file:
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@@
 <?xml version="1.0" encoding="utf-8"?>
 <!DOCTYPE eagle SYSTEM "eagle.dtd">
-<eagle version="9.3.0">
+<eagle version="9.2.2">
 <drawing>
 <settings>
@@
 <sheet>
 <plain>
-<text x="297.18" y="165.1" size="1.778" layer="94">Note: Short Jumper for open hi-hat
-Third pin of POT1 should be grounded</text>
+<text x="297.18" y="162.56" size="1.778" layer="94">Note:
+1) Short Jumper for open hi-hat
+2) Third pin of POT1 should be grounded</text>
 <text x="53.34" y="363.22" size="1.778" layer="94" rot="R180">Note: POT2B is grounded to AGND</text>
 <text x="149.86" y="76.2" size="1.778" layer="94">Note: R27 should be a jumper.
 The resistor is only there so biasing can be changed if needed.</text>
-<text x="241.3" y="205.74" size="1.778" layer="91">Note: used 330k</text>
-<text x="134.62" y="38.1" size="1.778" layer="91">used 2.2k</text>
+<text x="241.3" y="205.74" size="1.778" layer="94">Note: used 330k</text>
+<text x="119.38" y="27.94" size="1.778" layer="94">Note: used 2.2k since 2.7k
+was not available</text>
 <text x="7.62" y="411.48" size="6.4516" layer="94">24 Pin Header</text>
 <text x="73.66" y="411.48" size="6.4516" layer="94">Waveform Generator Input</text>
@@
 <net name="SQ_BUFFERED" class="0">
 <segment>
+<pinref part="J1" gate="G$1" pin="2"/>
+<wire x1="124.46" y1="391.16" x2="127" y2="391.16" width="0.1524" layer="91"/>
+<label x="128.016" y="387.858" size="1.778" layer="95"/>
 <pinref part="J1" gate="G$1" pin="4"/>
 <wire x1="124.46" y1="388.62" x2="127" y2="388.62" width="0.1524" layer="91"/>
-<label x="127" y="388.62" size="1.778" layer="95"/>
-</segment>
-<segment>
-<pinref part="J1" gate="G$1" pin="2"/>
-<wire x1="124.46" y1="391.16" x2="127" y2="391.16" width="0.1524" layer="91"/>
-<label x="127" y="391.16" size="1.778" layer="95"/>
-</segment>
-<segment>
+<wire x1="127" y1="391.16" x2="127" y2="388.62" width="0.1524" layer="91"/>
 <pinref part="J1" gate="G$1" pin="6"/>
 <wire x1="124.46" y1="386.08" x2="127" y2="386.08" width="0.1524" layer="91"/>
-<label x="127" y="386.08" size="1.778" layer="95"/>
+<wire x1="127" y1="388.62" x2="127" y2="386.08" width="0.1524" layer="91"/>
+<junction x="127" y="388.62"/>
 </segment>
 <segment>
@@
 <pinref part="J1" gate="G$1" pin="1"/>
 <wire x1="109.22" y1="391.16" x2="106.68" y2="391.16" width="0.1524" layer="91"/>
-<label x="88.9" y="391.16" size="1.778" layer="95"/>
-</segment>
-<segment>
+<label x="86.614" y="387.604" size="1.778" layer="95"/>
 <pinref part="J1" gate="G$1" pin="3"/>
 <wire x1="109.22" y1="388.62" x2="106.68" y2="388.62" width="0.1524" layer="91"/>
-<label x="88.9" y="388.62" size="1.778" layer="95"/>
-</segment>
-<segment>
+<wire x1="106.68" y1="391.16" x2="106.68" y2="388.62" width="0.1524" layer="91"/>
 <pinref part="J1" gate="G$1" pin="5"/>
 <wire x1="109.22" y1="386.08" x2="106.68" y2="386.08" width="0.1524" layer="91"/>
-<label x="88.9" y="386.08" size="1.778" layer="95"/>
-</segment>
-<segment>
+<wire x1="106.68" y1="388.62" x2="106.68" y2="386.08" width="0.1524" layer="91"/>
+<junction x="106.68" y="388.62"/>
+</segment>
+<segment>
