File: Power Supply/PCB/Power Supply.brd (EAGLE design)
At the start: 150 x 100 mm, 39 parts, among them IC1 LM741P, IC2 LM741P, IC3 LM741P

Commit message: Power supply PCB still in progress
Parts:
- added U$37, U$56, U$64: 100uF/50V, Capstone:100UF_CAP
- added U$38, U$57, U$58, U$65: 0.1uF/50V, Capstone:CERAMIC_CAPACITOR
- added U$39, U$45: 12V, Capstone:1W_ZENER
- added U$40, U$46: 500 OHM/0.5W, Capstone:0.5W_RES
- added U$41, U$42, U$47, U$48, U$60: 10k, Capstone:0.25W_RES
- added U$43, U$44, U$62, U$69: 1uF/50V, Capstone:CERAMIC_CAPACITOR
- added U$49: (no value), Capstone:DIODE-1N4001
- added U$50: 220uF/50V, Capstone:220UF_CAP
- added U$51: 1K/0.5W, Capstone:0.5W_RES
- added U$52, U$53: (no value), Capstone:TO-92
- added U$54: 10k, Capstone:10K_TRIM
- added U$55: 5k, Capstone:0.25W_RES
- added U$59: (no value), Capstone:10K_TRIM
- added U$61: 5.1V, Capstone:1W_ZENER
- added U$63: 2N4401, Capstone:TO-92
- added U$66: (no value), Capstone:TO220V
- added U$67: 6.2V, Capstone:1W_ZENER
- added U$68: 100 OHM, Capstone:0.25W_RES
- added U$70, U$71: P6KE15A-E3/54GICT-ND_TVS_DIODE, TVS Diode Through-Hole:P6KE15A-E3/54GICT-ND_TVS_DIODE
- U$10: value (none) -> 10 OHM/5W
- U$11: value (none) -> 1 OHM/5W
- U$16: value (none) -> 10000uF/16V
- U$30: value (none) -> 100uF/50V; device Capstone:220UF_CAP -> Capstone:100UF_CAP
- U$35: value (none) -> 10k
- U$36: value (none) -> 5k
- moved U$26 346.6 mm to (264.2, 175.3)
- moved U$27 346.6 mm to (264.2, 171.1)
- moved U$33 346.6 mm to (229.5, 168.0)
- moved U$34 346.6 mm to (223.9, 168.0)
- moved U$36 346.6 mm to (226.4, 158.0)
- moved U$3 133.5 mm to (1.34, 1.99), turned to 0 degrees
- moved U$2 131.6 mm to (51.8, 1.99), turned to 0 degrees
- moved U$1 103.7 mm to (83.1, 147.2), turned to 180 degrees
- moved U$14 85.6 mm to (1.80, 123.2), turned to 270 degrees
- moved U$15 85.6 mm to (26.6, 123.1), turned to 270 degrees
- moved U$17 85.3 mm to (14.2, 123.1), turned to 270 degrees
- moved U$12 52.1 mm to (45.3, 148.8)
- moved U$13 50.9 mm to (22.0, 148.9)
- moved U$16 47.2 mm to (13.3, 37.0), turned to 270 degrees
- moved U$5 45.3 mm to (37.1, 57.0), turned to 270 degrees
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Connections:
- removed net V+: IC2.7, IC3.7
- removed net V-: IC2.4, IC3.4
- new net +12V: IC3.7, U$3.P$3, U$36.P$2, U$37.P1+, U$38.P$1
- new net +12V_FEEDBACK: IC1.2, U$35.P$3, U$36.P$1
- new net +12V_REF: IC1.3, U$41.P$2, U$42.P$1
- new net +5V: U$1.P$3, U$59.P$3, U$64.P1+, U$65.P$1, U$67.P$2CATHODE
- new net +5V_FEEDBACK: IC3.2, U$59.P$2
- new net -12V: IC3.4, U$2.P$3, U$55.P$1, U$56.P2-, U$57.P$2
- new net -12V_FEEDBACK: IC2.2, U$54.P$2, U$55.P$2
- new net -12V_REF: IC2.3, U$47.P$1, U$48.P$2
- new net N$15: U$39.P$2CATHODE, U$40.P$1, U$42.P$2, U$43.P$1
- new net N$16: U$49.A, U$50.P2-, U$51.P$1, U$52.3
- new net N$17: IC3.3, U$60.P$1, U$61.P$2CATHODE, U$62.P$1
- new net N$18: U$44.P$2, U$45.P$1ANODE, U$46.P$2, U$48.P$1
- new net N$19: U$12.1, U$17.P$1
- new net N$20: U$30.P2-, U$51.P$2, U$52.2
- new net N$21: IC2.4, U$52.1
- new net N$23: U$10.P$2, U$2.P$2, U$53.3
- new net N$24: U$2.P$1, U$53.1
- new net N$25: IC2.6, U$53.2
- new net N$26: U$1.P$2, U$11.P$2, U$63.3
- new net N$27: U$12.2, U$24.A, U$25.C
- new net N$28: IC3.6, U$63.2
- new net N$29: U$22.C, U$24.C, U$7.P$1
- new net N$30: U$11.P$1, U$16.P1+, U$58.P$1, U$60.P$2, U$7.P$2
- new net N$32: U$1.P$1, U$63.1
- new net N$33: U$66.3, U$67.P$1ANODE, U$68.P$2, U$69.P$1
- new net OV_THYRISTOR: U$17.P$2, U$22.A, U$23.C, U$66.2
- net GND: now also IC2.7, U$16.P2-, U$23.A, U$25.A, U$30.P1+, U$35.P$2, U$37.P2-, U$38.P$2, U$39.P$1ANODE, U$41.P$1, U$43.P$2, U$44.P$1, U$45.P$2CATHODE, U$47.P$2, U$50.P1+, U$54.P$3, U$56.P1+, U$57.P$1, U$58.P$2, U$59.P$1, U$61.P$1ANODE, U$62.P$2, U$64.P2-, U$65.P$2, U$66.1, U$68.P$1, U$69.P$2
- net N$1: now also U$6.P$1; no longer U$14.P$1
- net N$2: now also U$14.P$2; no longer U$13.1
- net N$3: now also U$15.P$2; no longer U$13.3
- net N$4: now also U$8.P$1; no longer U$15.P$1
- net N$5: now also U$13.1, U$14.P$1; no longer U$14.P$2, U$6.P$1
- net N$6: now also U$13.3, U$15.P$1; no longer U$15.P$2, U$8.P$1
- net N$7: now also U$40.P$2
- net N$9: now also U$10.P$1, U$46.P$1, U$49.C
Other:
- board size 150 x 100 mm -> 100 x 150 mm

Commit message: Finished PCB
Parts:
- removed U$1: 60V/10A/25W, Capstone:TO-220_SMALL_HEATSINK
- removed U$10, U$9: 10 OHM/5W, Capstone:5W_RES
- removed U$11: 1 OHM/5W, Capstone:5W_RES
- removed U$12: (no value), Capstone:2_PIN_CONNECT
- removed U$13: (no value), Capstone:3_PIN_TE
- removed U$14, U$15, U$17: (no value), Capstone:FUSEHOLDER
- removed U$16: 10000uF/16V, Capstone:POLARIZED_CAP_3300UF
- removed U$18, U$19, U$20, U$21, U$22, U$23, U$24, U$25, U$28, U$49: (no value), Capstone:DIODE-1N4001
- removed U$2, U$3: 100V/3A/40W, Capstone:TO-220_LARGE_HEATSINK
- removed U$26, U$27, U$38, U$57, U$58, U$65: 0.1uF/50V, Capstone:CERAMIC_CAPACITOR
- removed U$29, U$50: 220uF/50V, Capstone:220UF_CAP
- removed U$30, U$31, U$37, U$56, U$64: 100uF/50V, Capstone:100UF_CAP
- removed U$32, U$51: 1K/0.5W, Capstone:0.5W_RES
- removed U$33, U$34, U$52, U$53: (no value), Capstone:TO-92
- removed U$35, U$54: 10k, Capstone:10K_TRIM
- removed U$36, U$55: 5k, Capstone:0.25W_RES
- removed U$39, U$45: 12V, Capstone:1W_ZENER
- removed U$4, U$5: 3300uF/50V, Capstone:POLARIZED_CAP_3300UF
- removed U$40, U$46: 500 OHM/0.5W, Capstone:0.5W_RES
- removed U$41, U$42, U$47, U$48, U$60: 10k, Capstone:0.25W_RES
- removed U$43, U$44, U$62, U$69: 1uF/50V, Capstone:CERAMIC_CAPACITOR
- removed U$59: (no value), Capstone:10K_TRIM
- removed U$6, U$7, U$8: 47uH/2.3A, Capstone:47UH_2.3A_COIL
- removed U$61: 5.1V, Capstone:1W_ZENER
- removed U$63: 2N4401, Capstone:TO-92
- removed U$66: (no value), Capstone:TO220V
- removed U$67: 6.2V, Capstone:1W_ZENER
- removed U$68: 100 OHM, Capstone:0.25W_RES
- removed U$70, U$71: P6KE15A-E3/54GICT-ND_TVS_DIODE, TVS Diode Through-Hole:P6KE15A-E3/54GICT-ND_TVS_DIODE
- added 33V: (no value), Capstone:3_PIN_TE
- added 6.3V: (no value), Capstone:2_PIN_CONNECT
- added C1, C11, C16, C19, C2, C5: 0.1uF/50V, Capstone:CERAMIC_CAPACITOR
- added C10, C14, C15, C18, C9: 100uF/50V, Capstone:100UF_CAP
- added C12, C17, C20, C7: 1uF/50V, Capstone:CERAMIC_CAPACITOR
- added C13, C8: 220uF/50V, Capstone:220UF_CAP
- added C3, C4: 3300uF/50V, Capstone:POLARIZED_CAP_3300UF
- added C6: 10000uF/16V, Capstone:POLARIZED_CAP_3300UF
- added D1, D10, D12, D2, D3, D4, D5, D6, D7, D8: (no value), Capstone:DIODE-1N4001
- added D11, D9: 12V, Capstone:1W_ZENER
- added D13: 5.1V, Capstone:1W_ZENER
- added D14: 6.2V, Capstone:1W_ZENER
- added F1, F2, F3: (no value), Capstone:FUSEHOLDER
- added GND: M3_SCREW_TERMINAL, EcoCar Temp:M3_SCREW_TERMINAL
- added H1, H2, H3, H4: STAND-OFF, SparkFun-Hardware:STAND-OFF
- added L1, L2, L3: 47uH/2.3A, Capstone:47UH_2.3A_COIL
- added POWER_1, POWER_2, POWER_3, POWER_4, POWER_5, POWER_6, POWER_7: TE-6PIN, Capstone:TE_6_PIN
- added Q1, Q2, Q4, Q5: (no value), Capstone:TO-92
- added Q3, Q6: 100V/3A/40W, Capstone:TO-220_LARGE_HEATSINK
- added Q7: 2N4401, Capstone:TO-92
- added Q8: 60V/10A/25W, Capstone:TO-220_SMALL_HEATSINK
- added R1, R9: 500 OHM/0.5W, Capstone:0.5W_RES
- added R10, R5: 1K/0.5W, Capstone:0.5W_RES
- added R11, R4: 10 OHM/5W, Capstone:5W_RES
- added R12, R6: 5k, Capstone:0.25W_RES
- added R13, R2, R3, R7, R8: 10k, Capstone:0.25W_RES
- added R14: 1 OHM/5W, Capstone:5W_RES
- added R15: 100 OHM, Capstone:0.25W_RES
- added SCR1: (no value), Capstone:TO220V
- added TRIM1, TRIM2: 10k, Capstone:10K_TRIM
- added TRIM3: (no value), Capstone:10K_TRIM
- IC1, IC2, IC3: value LM741P -> LM741; device linear:DIL08 -> Capstone:DIL08
- moved IC3 108.6 mm to (86.0, 141.0)
- moved IC2 34.9 mm to (88.0, 43.0)
- moved IC1 4.32 mm to (57.6, 27.8)
Connections:
- net +12V: now also C10.P1+, C11.P$1, POWER_1.4, POWER_2.4, POWER_3.4, POWER_4.4, POWER_5.4, POWER_6.4, POWER_7.4, Q3.P$3, R6.P$2; no longer U$3.P$3, U$36.P$2, U$37.P1+, U$38.P$1
- net +12V_FEEDBACK: now also R6.P$1, TRIM1.P$3; no longer U$35.P$3, U$36.P$1
- net +12V_REF: now also R2.P$1, R3.P$2; no longer U$41.P$2, U$42.P$1
- net +5V: now also C18.P1+, C19.P$1, D14.P$2CATHODE, POWER_1.6, POWER_2.6, POWER_3.6, POWER_4.6, POWER_5.6, POWER_6.6, POWER_7.6, Q8.P$3, TRIM3.P$3; no longer U$1.P$3, U$59.P$3, U$64.P1+, U$65.P$1, U$67.P$2CATHODE
- net +5V_FEEDBACK: now also TRIM3.P$2; no longer U$59.P$2
- net -12V: now also C15.P2-, C16.P$2, POWER_1.5, POWER_2.5, POWER_3.5, POWER_4.5, POWER_5.5, POWER_6.5, POWER_7.5, Q6.P$3, R12.P$1; no longer U$2.P$3, U$55.P$1, U$56.P2-, U$57.P$2
- net -12V_FEEDBACK: now also R12.P$2, TRIM2.P$2; no longer U$54.P$2, U$55.P$2
- net -12V_REF: now also R7.P$1, R8.P$2; no longer U$47.P$1, U$48.P$2
- net GND: now also 33V.2, C1.P$2, C10.P2-, C11.P$2, C12.P$1, C13.P1+, C14.P1+, C15.P1+, C16.P$1, C17.P$2, C18.P2-, C19.P$2, C2.P$1, C20.P$2, C3.P2-, C4.P1+, C5.P$2, C6.P2-, C7.P$2, C8.P2-, C9.P2-, D11.P$2CATHODE, D13.P$1ANODE, D6.A, D8.A, D9.P$1ANODE, GND.1, GND.2, GND.3, GND.4, POWER_1.1, POWER_1.2, POWER_1.3, POWER_2.1, POWER_2.2, POWER_2.3, POWER_3.1, POWER_3.2, POWER_3.3, POWER_4.1, POWER_4.2, POWER_4.3, POWER_5.1, POWER_5.2, POWER_5.3, POWER_6.1, POWER_6.2, POWER_6.3, POWER_7.1, POWER_7.2, POWER_7.3, R15.P$1, R3.P$1, R7.P$2, SCR1.1, TRIM1.P$2, TRIM2.P$3, TRIM3.P$1; no longer U$13.2, U$16.P2-, U$23.A, U$25.A, U$26.P$2, U$27.P$1, U$29.P2-, U$30.P1+, U$31.P2-, U$35.P$2, U$37.P2-, U$38.P$2, U$39.P$1ANODE, U$4.P2-, U$41.P$1, U$43.P$2, U$44.P$1, U$45.P$2CATHODE, U$47.P$2, U$5.P1+, U$50.P1+, U$54.P$3, U$56.P1+, U$57.P$1, U$58.P$2, U$59.P$1, U$61.P$1ANODE, U$62.P$2, U$64.P2-, U$65.P$2, U$66.1, U$68.P$1, U$69.P$2
- net N$1: now also D1.C, D3.C, L1.P$1; no longer U$18.C, U$20.C, U$6.P$1
- net N$10: now also C9.P1+, Q1.2, R5.P$1; no longer U$31.P1+, U$32.P$1, U$33.2
- net N$11: now also Q1.1; no longer U$33.1
- net N$12: now also Q2.3, Q3.P$2, R4.P$2; no longer U$3.P$2, U$34.3, U$9.P$2
- net N$13: now also Q2.1, Q3.P$1; no longer U$3.P$1, U$34.1
- net N$14: now also Q2.2; no longer U$34.2
- net N$15: now also C7.P$1, D9.P$2CATHODE, R1.P$1, R2.P$2; no longer U$39.P$2CATHODE, U$40.P$1, U$42.P$2, U$43.P$1
- net N$16: now also C13.P2-, D12.A, Q4.3, R10.P$1; no longer U$49.A, U$50.P2-, U$51.P$1, U$52.3
- net N$17: now also C17.P$1, D13.P$2CATHODE, R13.P$1; no longer U$60.P$1, U$61.P$2CATHODE, U$62.P$1
- net N$18: now also C12.P$2, D11.P$1ANODE, R8.P$1, R9.P$2; no longer U$44.P$2, U$45.P$1ANODE, U$46.P$2, U$48.P$1
- net N$19: now also 6.3V.1, F3.P$1; no longer U$12.1, U$17.P$1
- net N$2: now also D1.A, D2.C, F1.P$2; no longer U$14.P$2, U$18.A, U$19.C
- net N$20: now also C14.P2-, Q4.2, R10.P$2; no longer U$30.P2-, U$51.P$2, U$52.2
- net N$21: now also Q4.1; no longer U$52.1
- net N$23: now also Q5.3, Q6.P$2, R11.P$2; no longer U$10.P$2, U$2.P$2, U$53.3
- net N$24: now also Q5.1, Q6.P$1; no longer U$2.P$1, U$53.1
- net N$25: now also Q5.2; no longer U$53.2
- net N$26: now also Q7.3, Q8.P$2, R14.P$2; no longer U$1.P$2, U$11.P$2, U$63.3
- net N$27: now also 6.3V.2, D7.A, D8.C; no longer U$12.2, U$24.A, U$25.C
- net N$28: now also Q7.2; no longer U$63.2
- net N$29: now also D5.C, D7.C, L3.P$1; no longer U$22.C, U$24.C, U$7.P$1
- net N$3: now also D3.A, D4.C, F2.P$2; no longer U$15.P$2, U$20.A, U$21.C
- net N$30: now also C5.P$1, C6.P1+, L3.P$2, R13.P$2, R14.P$1; no longer U$11.P$1, U$16.P1+, U$58.P$1, U$60.P$2, U$7.P$2
- net N$32: now also Q7.1, Q8.P$1; no longer U$1.P$1, U$63.1
- net N$33: now also C20.P$1, D14.P$1ANODE, R15.P$2, SCR1.3; no longer U$66.3, U$67.P$1ANODE, U$68.P$2, U$69.P$1
- net N$4: now also D2.A, D4.A, L2.P$1; no longer U$19.A, U$21.A, U$8.P$1
- net N$5: now also 33V.1, F1.P$1; no longer U$13.1, U$14.P$1
- net N$6: now also 33V.3, F2.P$1; no longer U$13.3, U$15.P$1
- net N$7: now also C1.P$1, C3.P1+, D10.A, L1.P$2, R1.P$2, R4.P$1; no longer U$26.P$1, U$28.A, U$4.P1+, U$40.P$2, U$6.P$2, U$9.P$1
- net N$8: now also C8.P1+, D10.C, Q1.3, R5.P$2; no longer U$28.C, U$29.P1+, U$32.P$2, U$33.3
- net N$9: now also C2.P$2, C4.P2-, D12.C, L2.P$2, R11.P$1, R9.P$1; no longer U$10.P$1, U$27.P$2, U$46.P$1, U$49.C, U$5.P2-, U$8.P$2
- net OV_THYRISTOR: now also D5.A, D6.C, F3.P$2, SCR1.2; no longer U$17.P$2, U$22.A, U$23.C, U$66.2
Routing:
- net GND: track 0.00 -> 1182.0 mm, vias 0 -> 5
- net +12V: track 0.00 -> 417.2 mm, vias 0 -> 2
- net -12V: track 0.00 -> 374.5 mm
- net +5V: track 0.00 -> 261.2 mm, vias 0 -> 15
- net N$30: track 0.00 -> 86.8 mm, vias 0 -> 2
- net N$9: track 0.00 -> 84.9 mm
- net N$7: track 0.00 -> 67.6 mm
- net N$27: track 0.00 -> 66.4 mm
- net N$24: track 0.00 -> 65.4 mm, vias 0 -> 1
- net N$21: track 0.00 -> 60.2 mm, vias 0 -> 1
- net N$5: track 0.00 -> 56.6 mm
- net N$23: track 0.00 -> 54.8 mm
- net OV_THYRISTOR: track 0.00 -> 52.1 mm
- net N$12: track 0.00 -> 42.1 mm
- net N$28: track 0.00 -> 41.0 mm
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Other:
- board size 100 x 150 mm -> 120 x 150 mm
- board text added: "GND"
- board text added: "Power Supply V1.0"

Commit message: updated schematic
Parts:
- D1, D10, D12, D2, D3, D4, D5, D6, D7, D8: value (none) -> 1N4005
- D13: value 5.1V -> 3.3V
- F1, F2: value (none) -> 500mA Slow Blow
- F3: value (none) -> 750mA Slow Blow
- Q1, Q2: value (none) -> 2N4401
- Q4, Q5: value (none) -> 2N4403
- R13: value 10k -> 100
Changed lines of the file:
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@@
 <?xml version="1.0" encoding="utf-8"?>
 <!DOCTYPE eagle SYSTEM "eagle.dtd">
-<eagle version="8.6.2">
+<eagle version="9.2.2">
 <drawing>
 <settings>
@@
 <param name="checkStop" value="0"/>
 <param name="checkValues" value="0"/>
+<param name="checkNames" value="1"/>
+<param name="checkWireStubs" value="1"/>
+<param name="checkPolygonWidth" value="0"/>
 <param name="useDiameter" value="13"/>
 <param name="maxErrors" value="50"/>
@@
 <attribute name="NAME" x="49.4" y="133.09" size="1.778" layer="25" rot="R180"/>
 </element>
-<element name="F1" library="Capstone" package="FUSEHOLDER" value="" x="2" y="128.1" smashed="yes" rot="R270">
+<element name="F1" library="Capstone" package="FUSEHOLDER" value="500mA Slow Blow" x="2" y="128.1" smashed="yes" rot="R270">
 <attribute name="NAME" x="11.865" y="127.827" size="1.778" layer="25" rot="R270"/>
 <attribute name="VALUE" x="12.5" y="114.3" size="1.778" layer="27" rot="R270"/>
 </element>
-<element name="F2" library="Capstone" package="FUSEHOLDER" value="" x="14.6" y="128.1" smashed="yes" rot="R270">
+<element name="F2" library="Capstone" package="FUSEHOLDER" value="500mA Slow Blow" x="14.6" y="128.1" smashed="yes" rot="R270">
 <attribute name="NAME" x="24.465" y="127.954" size="1.778" layer="25" rot="R270"/>
 <attribute name="VALUE" x="25.1" y="114.3" size="1.778" layer="27" rot="R270"/>
 </element>
-<element name="F3" library="Capstone" package="FUSEHOLDER" value="" x="27.2" y="128.1" smashed="yes" rot="R270">
+<element name="F3" library="Capstone" package="FUSEHOLDER" value="750mA Slow Blow" x="27.2" y="128.1" smashed="yes" rot="R270">
 <attribute name="NAME" x="37.192" y="127.827" size="1.778" layer="25" rot="R270"/>
 <attribute name="VALUE" x="37.7" y="114.3" size="1.778" layer="27" rot="R270"/>
 </element>
-<element name="D1" library="Capstone" package="DIODE-1N4001" value="" x="18" y="94" smashed="yes" rot="R270">
+<element name="D1" library="Capstone" package="DIODE-1N4001" value="1N4005" x="18" y="94" smashed="yes" rot="R270">
 <attribute name="NAME" x="15.714" y="94" size="0.6096" layer="25" font="vector" ratio="20" rot="R270" align="bottom-center"/>
 </element>
-<element name="D2" library="Capstone" package="DIODE-1N4001" value="" x="13" y="94" smashed="yes" rot="R90">
+<element name="D2" library="Capstone" package="DIODE-1N4001" value="1N4005" x="13" y="94" smashed="yes" rot="R90">
 <attribute name="NAME" x="11.349" y="94.011" size="0.6096" layer="25" font="vector" ratio="20" rot="R90" align="bottom-center"/>
 </element>
-<element name="D3" library="Capstone" package="DIODE-1N4001" value="" x="8" y="94" smashed="yes" rot="R270">
+<element name="D3" library="Capstone" package="DIODE-1N4001" value="1N4005" x="8" y="94" smashed="yes" rot="R270">
 <attribute name="NAME" x="5.841" y="94" size="0.6096" layer="25" font="vector" ratio="20" rot="R270" align="bottom-center"/>
 </element>
-<element name="D4" library="Capstone" package="DIODE-1N4001" value="" x="3" y="94" smashed="yes" rot="R90">
+<element name="D4" library="Capstone" package="DIODE-1N4001" value="1N4005" x="3" y="94" smashed="yes" rot="R90">
 <attribute name="NAME" x="1.476" y="94" size="0.6096" layer="25" font="vector" ratio="20" rot="R90" align="bottom-center"/>
 </element>
-<element name="D5" library="Capstone" package="DIODE-1N4001" value="" x="38" y="94" smashed="yes" rot="R270">
+<element name="D5" library="Capstone" package="DIODE-1N4001" value="1N4005" x="38" y="94" smashed="yes" rot="R270">
 <attribute name="NAME" x="35.841" y="94" size="0.6096" layer="25" font="vector" ratio="20" rot="R270" align="bottom-center"/>
 </element>
-<element name="D6" library="Capstone" package="DIODE-1N4001" value="" x="33" y="94" smashed="yes" rot="R90">
+<element name="D6" library="Capstone" package="DIODE-1N4001" value="1N4005" x="33" y="94" smashed="yes" rot="R90">
 <attribute name="NAME" x="31.476" y="94" size="0.6096" layer="25" font="vector" ratio="20" rot="R90" align="bottom-center"/>
 </element>
-<element name="D7" library="Capstone" package="DIODE-1N4001" value="" x="28" y="94" smashed="yes" rot="R270">
+<element name="D7" library="Capstone" package="DIODE-1N4001" value="1N4005" x="28" y="94" smashed="yes" rot="R270">
 <attribute name="NAME" x="25.714" y="94" size="0.6096" layer="25" font="vector" ratio="20" rot="R270" align="bottom-center"/>
 </element>
-<element name="D8" library="Capstone" package="DIODE-1N4001" value="" x="23" y="94" smashed="yes" rot="R90">
+<element name="D8" library="Capstone" package="DIODE-1N4001" value="1N4005" x="23" y="94" smashed="yes" rot="R90">
 <attribute name="NAME" x="21.476" y="94" size="0.6096" layer="25" font="vector" ratio="20" rot="R90" align="bottom-center"/>
 </element>
@@
 <attribute name="NAME" x="64.748" y="80.69" size="1.016" layer="25"/>
 </element>
-<element name="D10" library="Capstone" package="DIODE-1N4001" value="" x="53.704" y="61.8" smashed="yes">
+<element name="D10" library="Capstone" package="DIODE-1N4001" value="1N4005" x="53.704" y="61.8" smashed="yes">
 <attribute name="NAME" x="53.704" y="63.324" size="0.6096" layer="25" font="vector" ratio="20" align="bottom-center"/>
 </element>
@@
 <attribute name="NAME" x="53.224" y="58.738" size="0.6096" layer="25"/>
 </element>
-<element name="Q1" library="Capstone" package="TO-92" value="" x="57.5648" y="39.5" smashed="yes">
+<element name="Q1" library="Capstone" package="TO-92" value="2N4401" x="57.5648" y="39.5" smashed="yes">
 <attribute name="NAME" x="57.5648" y="42.548" size="0.6096" layer="25" font="vector" ratio="20" align="bottom-center"/>
 </element>
-<element name="Q2" library="Capstone" package="TO-92" value="" x="41" y="27.9" smashed="yes" rot="R270">
+<element name="Q2" library="Capstone" package="TO-92" value="2N4401" x="41" y="27.9" smashed="yes" rot="R270">
 <attribute name="NAME" x="44.048" y="27.9" size="0.6096" layer="25" font="vector" ratio="20" rot="R270" align="bottom-center"/>
 </element>
@@
 <attribute name="NAME" x="83.876" y="55.762" size="0.6096" layer="25" rot="R180"/>
 </element>
-<element name="D12" library="Capstone" package="DIODE-1N4001" value="" x="69.7" y="84" smashed="yes" rot="R180">
+<element name="D12" library="Capstone" package="DIODE-1N4001" value="1N4005" x="69.7" y="84" smashed="yes" rot="R180">
 <attribute name="NAME" x="69.7" y="82.476" size="0.6096" layer="25" font="vector" ratio="20" rot="R180" align="bottom-center"/>
 </element>
@@
 <attribute name="NAME" x="81.624" y="100.438" size="0.6096" layer="25"/>
 </element>
-<element name="Q4" library="Capstone" package="TO-92" value="" x="83.2" y="84" smashed="yes" rot="R180">
+<element name="Q4" library="Capstone" package="TO-92" value="2N4403" x="83.2" y="84" smashed="yes" rot="R180">
 <attribute name="NAME" x="83.2" y="80.952" size="0.6096" layer="25" font="vector" ratio="20" rot="R180" align="bottom-center"/>
 </element>
-<element name="Q5" library="Capstone" package="TO-92" value="" x="77.703" y="38.049" smashed="yes" rot="R180">
+<element name="Q5" library="Capstone" package="TO-92" value="2N4403" x="77.703" y="38.049" smashed="yes" rot="R180">
 <attribute name="NAME" x="77.703" y="35.001" size="0.6096" layer="25" font="vector" ratio="20" rot="R180" align="bottom-center"/>
 </element>
@@
 <attribute name="NAME" x="84.914" y="111.555" size="1.016" layer="25" rot="R180"/>
 </element>
-<element name="R13" library="Capstone" package="0.25W_RES" value="10k" x="81.57813125" y="124.5" smashed="yes" rot="R270">
+<element name="R13" library="Capstone" package="0.25W_RES" value="100" x="81.57813125" y="124.5" smashed="yes" rot="R270">
 <attribute name="NAME" x="82.71613125" y="125.876" size="0.6096" layer="25" rot="R270"/>
 </element>
-<element name="D13" library="Capstone" package="1W_ZENER" value="5.1V" x="91.19999375" y="124.5" smashed="yes" rot="R90">
+<element name="D13" library="Capstone" package="1W_ZENER" value="3.3V" x="91.19999375" y="124.5" smashed="yes" rot="R90">
 <attribute name="NAME" x="90.05699375" y="122.468" size="0.8128" layer="25" rot="R90"/>
 </element>
@@
 </signal>
 </signals>
+<mfgpreviewcolors>
+<mfgpreviewcolor name="soldermaskcolor" color="0xC8008000"/>
+<mfgpreviewcolor name="silkscreencolor" color="0xFFFEFEFE"/>
+<mfgpreviewcolor name="backgroundcolor" color="0xFF282828"/>
+<mfgpreviewcolor name="coppercolor" color="0xFFFFBF00"/>
+<mfgpreviewcolor name="substratecolor" color="0xFF786E46"/>
+</mfgpreviewcolors>
 </board>
 </drawing>
